Commit message: Fixed the launch script.

File: adabot.xacro (robot description, xacro)
@@ -22,4 +22,13 @@
     </material>
     <!--
+         Macro for creating wheel geoms
+    -->
+    <xacro:property name="wh-geom">
+        <origin rpy="1.57075 0 0" xyz="0 0 0" />
+        <geometry>
+            <cylinder radius="${wh_radius}" length="${wh_length}" />
+        </geometry>
+    </xacro:property>
+    <!--
          Macro for creating wheels
     -->
@@ -27,14 +36,16 @@
         <link name="wh-${suffix}">
             <visual>
+                <xacro:insert_block name="wh-geom" />
+                <material name="black" />
+                <origin rpy="1.57075 0 0" xyz="0 0 0" />
+            </visual>
+            <collision>
+                <xacro:insert_block name="wh-geom" />
                 <geometry>
-                    <cylinder radius="${wh_radius}" length="${wh_length}" />
-                </geometry>
-                <material name="black" />
-            </visual>
         </link>
-        <joint name="ax-${suffix}" type="fixed">
+        <joint name="ax-${suffix}" type="continuous">
             <parent link="${parent}" />
             <child link="wh-${suffix}" />
-            <origin xyz="${ch_length/2*reflect_fb} ${ch_width/2*reflect_lr} ${zoffset}" rpy="0 1.57 0" />
+            <origin rpy="0 0 0 " xyz="${ch_length/2*reflect_fb} ${(wh_length+ch_width)/2*reflect_lr} ${zoffset}" />
             <axis xyz="${ax_axis}" />
         </joint>

File: src/adabot_description/urdf/adabot.urdf (robot description, URDF)
Before this commit: robot adabot, 5 links, 4 joints
Joints:
- joint ax-back-left: origin xyz=-1.0 -1.0 0.275 rpy=0 1.57 0 -> xyz=-1.0 -1.0 0.275 rpy=0 0 0 ; type fixed -> continuous
- joint ax-back-right: origin xyz=-1.0 1.0 0.275 rpy=0 1.57 0 -> xyz=-1.0 1.0 0.275 rpy=0 0 0 ; type fixed -> continuous
- joint ax-front-left: origin xyz=1.0 -1.0 0.275 rpy=0 1.57 0 -> xyz=1.0 -1.0 0.275 rpy=0 0 0 ; type fixed -> continuous
- joint ax-front-right: origin xyz=1.0 1.0 0.275 rpy=0 1.57 0 -> xyz=1.0 1.0 0.275 rpy=0 0 0 ; type fixed -> continuous

Commit message: Xacro file is in a semi-complete state (proper sizes and all required attributes are correct).

File: adabot.xacro (robot description, xacro)
@@ -4,10 +4,12 @@
          Properties for the geometries
     -->
-    <xacro:property name="wh_radius" value="0.5" />
-    <xacro:property name="wh_length" value="0.2" />
+    <xacro:property name="wh_radius" value="0.02" />
+    <xacro:property name="wh_length" value="0.005" />
+    <xacro:property name="wh_mass" value="${500*3.145927*(wh_radius**2)*wh_length}" />
     <xacro:property name="ax_axis" value="0 1 0" />
-    <xacro:property name="ch_length" value="2" />
-    <xacro:property name="ch_width" value="2" />
-    <xacro:property name="ch_height" value="0.5" />
+    <xacro:property name="ch_length" value="0.1" />
+    <xacro:property name="ch_width" value="0.07" />
+    <xacro:property name="ch_height" value="0.035" />
+    <xacro:property name="ch_mass" value="${500*ch_length*ch_width*ch_height}" />
     <xacro:property name="zoffset" value="${wh_radius*1.1/2}" />
     <!--
@@ -24,5 +26,5 @@
          Macro for creating wheel geoms
     -->
-    <xacro:property name="wh-geom">
+    <xacro:property name="wh_orig_geom">
         <origin rpy="1.57075 0 0" xyz="0 0 0" />
         <geometry>
@@ -36,11 +38,21 @@
         <link name="wh-${suffix}">
             <visual>
-                <xacro:insert_block name="wh-geom" />
+                <xacro:insert_block name="wh_orig_geom" />
                 <material name="black" />
-                <origin rpy="1.57075 0 0" xyz="0 0 0" />
             </visual>
             <collision>
-                <xacro:insert_block name="wh-geom" />
-                <geometry>
+                <xacro:insert_block name="wh_orig_geom" />
+            </collision>
+            <inertial>
+                <mass value="${wh_mass}" />
+                <inertia
+                    ixx="${(1/12)*wh_mass*(3*wh_radius**2 + wh_length**2)}"
+                    ixy="0"
+                    ixz="0"
+                    iyy="${(1/12)*wh_mass*(3*wh_radius**2 + wh_length**2)}"
+                    iyz="0"
+                    izz="${(1/2)*wh_mass*wh_radius**2}"
+                    />
+            </inertial>
         </link>
         <joint name="ax-${suffix}" type="continuous">
@@ -52,14 +64,34 @@
     </xacro:macro>
     <!--
+         Macro for creating the chassis' geom
+    -->
+    <xacro:property name="ch_orig_geom">
+        <origin rpy="0 0 0" xyz="0 0 ${zoffset}" />
+        <geometry>
+            <box size="${ch_length} ${ch_width} ${ch_height}" />
+        </geometry>
+    </xacro:property>
+    <!--
          The main chassis/body
     -->
     <link name="${chassisname}">
         <visual>
-            <geometry>
-                <box size="${ch_length} ${ch_width} ${ch_height}" />
-            </geometry>
-            <origin rpy="0 0 0" xyz="0 0 ${zoffset}" />
+            <xacro:insert_block name="ch_orig_geom" />
             <material name="white" />
         </visual>
+        <collision>
+            <xacro:insert_block name="ch_orig_geom" />
+        </collision>
+        <inertial>
+            <mass value="${ch_mass}" />
+            <inertia
+                ixx="${(1/12)*ch_mass*(ch_width**2 + ch_height**2)}"
+                ixy="0"
+                ixz="0"
+                iyy="${(1/12)*ch_mass*(ch_length**2 + ch_height**2)}"
+                iyz="0"
+                izz="${(1/12)*ch_mass*(ch_length**2 + ch_width**2)}"
+                />
+        </inertial>
     </link>
     <!--

File: src/adabot_description/urdf/adabot.urdf (robot description, URDF)
Before this commit: robot adabot, 5 links, 4 joints
Links:
- link base_link: mass None -> 0.1225; geometry collision box size=0.1 0.07 0.035; visual box size=0.1 0.07 0.035
- link wh-back-left: mass None -> 0.003145927; geometry collision cylinder length=0.005 radius=0.02; visual cylinder length=0.005 radius=0.02
- link wh-back-right: mass None -> 0.003145927; geometry collision cylinder length=0.005 radius=0.02; visual cylinder length=0.005 radius=0.02
- link wh-front-left: mass None -> 0.003145927; geometry collision cylinder length=0.005 radius=0.02; visual cylinder length=0.005 radius=0.02
- link wh-front-right: mass None -> 0.003145927; geometry collision cylinder length=0.005 radius=0.02; visual cylinder length=0.005 radius=0.02
Joints:
- joint ax-back-left: origin xyz=-1.0 -1.0 0.275 rpy=0 0 0  -> xyz=-0.05 -0.0375 0.011 rpy=0 0 0 
- joint ax-back-right: origin xyz=-1.0 1.0 0.275 rpy=0 0 0  -> xyz=-0.05 0.0375 0.011 rpy=0 0 0 
- joint ax-front-left: origin xyz=1.0 -1.0 0.275 rpy=0 0 0  -> xyz=0.05 -0.0375 0.011 rpy=0 0 0 
- joint ax-front-right: origin xyz=1.0 1.0 0.275 rpy=0 0 0  -> xyz=0.05 0.0375 0.011 rpy=0 0 0 
