Commit message: Added wegs to .xacro file

File: src/adabot_description/urdf/adabot.urdf (robot description, URDF)
Before this commit: robot adabot, 5 links, 4 joints
Links:
- added link wg-back-left-1, mass 4e-05; collision box size=0.002 0.001 0.04; visual box size=0.002 0.001 0.04
- added link wg-back-left-2, mass 4e-05; collision box size=0.002 0.001 0.04; visual box size=0.002 0.001 0.04
- added link wg-back-left-3, mass 4e-05; collision box size=0.002 0.001 0.04; visual box size=0.002 0.001 0.04
- added link wg-back-left-4, mass 4e-05; collision box size=0.002 0.001 0.04; visual box size=0.002 0.001 0.04
- added link wg-back-left-5, mass 4e-05; collision box size=0.002 0.001 0.04; visual box size=0.002 0.001 0.04
- added link wg-back-right-1, mass 4e-05; collision box size=0.002 0.001 0.04; visual box size=0.002 0.001 0.04
- added link wg-back-right-2, mass 4e-05; collision box size=0.002 0.001 0.04; visual box size=0.002 0.001 0.04
- added link wg-back-right-3, mass 4e-05; collision box size=0.002 0.001 0.04; visual box size=0.002 0.001 0.04
- added link wg-back-right-4, mass 4e-05; collision box size=0.002 0.001 0.04; visual box size=0.002 0.001 0.04
- added link wg-back-right-5, mass 4e-05; collision box size=0.002 0.001 0.04; visual box size=0.002 0.001 0.04
- added link wg-front-left-1, mass 4e-05; collision box size=0.002 0.001 0.04; visual box size=0.002 0.001 0.04
- added link wg-front-left-2, mass 4e-05; collision box size=0.002 0.001 0.04; visual box size=0.002 0.001 0.04
- added link wg-front-left-3, mass 4e-05; collision box size=0.002 0.001 0.04; visual box size=0.002 0.001 0.04
- added link wg-front-left-4, mass 4e-05; collision box size=0.002 0.001 0.04; visual box size=0.002 0.001 0.04
- added link wg-front-left-5, mass 4e-05; collision box size=0.002 0.001 0.04; visual box size=0.002 0.001 0.04
- added link wg-front-right-1, mass 4e-05; collision box size=0.002 0.001 0.04; visual box size=0.002 0.001 0.04
- added link wg-front-right-2, mass 4e-05; collision box size=0.002 0.001 0.04; visual box size=0.002 0.001 0.04
- added link wg-front-right-3, mass 4e-05; collision box size=0.002 0.001 0.04; visual box size=0.002 0.001 0.04
- added link wg-front-right-4, mass 4e-05; collision box size=0.002 0.001 0.04; visual box size=0.002 0.001 0.04
- added link wg-front-right-5, mass 4e-05; collision box size=0.002 0.001 0.04; visual box size=0.002 0.001 0.04
Joints:
- added joint wg-back-left-1-joint: type prismatic, parent wh-back-left, child wg-back-left-1, origin xyz=0 0 0 rpy=0 1.25663706144 0, limit lower=0.005 upper=0 effort=1 velocity=1
- added joint wg-back-left-2-joint: type prismatic, parent wh-back-left, child wg-back-left-2, origin xyz=0 0 0 rpy=0 2.51327412287 0, limit lower=0.005 upper=0 effort=1 velocity=1
- added joint wg-back-left-3-joint: type prismatic, parent wh-back-left, child wg-back-left-3, origin xyz=0 0 0 rpy=0 3.76991118431 0, limit lower=0.005 upper=0 effort=1 velocity=1
- added joint wg-back-left-4-joint: type prismatic, parent wh-back-left, child wg-back-left-4, origin xyz=0 0 0 rpy=0 5.02654824574 0, limit lower=0.005 upper=0 effort=1 velocity=1
- added joint wg-back-left-5-joint: type prismatic, parent wh-back-left, child wg-back-left-5, origin xyz=0 0 0 rpy=0 6.28318530718 0, limit lower=0.005 upper=0 effort=1 velocity=1
- added joint wg-back-right-1-joint: type prismatic, parent wh-back-right, child wg-back-right-1, origin xyz=0 0 0 rpy=0 1.25663706144 0, limit lower=0.005 upper=0 effort=1 velocity=1
- added joint wg-back-right-2-joint: type prismatic, parent wh-back-right, child wg-back-right-2, origin xyz=0 0 0 rpy=0 2.51327412287 0, limit lower=0.005 upper=0 effort=1 velocity=1
- added joint wg-back-right-3-joint: type prismatic, parent wh-back-right, child wg-back-right-3, origin xyz=0 0 0 rpy=0 3.76991118431 0, limit lower=0.005 upper=0 effort=1 velocity=1
- added joint wg-back-right-4-joint: type prismatic, parent wh-back-right, child wg-back-right-4, origin xyz=0 0 0 rpy=0 5.02654824574 0, limit lower=0.005 upper=0 effort=1 velocity=1
- added joint wg-back-right-5-joint: type prismatic, parent wh-back-right, child wg-back-right-5, origin xyz=0 0 0 rpy=0 6.28318530718 0, limit lower=0.005 upper=0 effort=1 velocity=1
- added joint wg-front-left-1-joint: type prismatic, parent wh-front-left, child wg-front-left-1, origin xyz=0 0 0 rpy=0 1.25663706144 0, limit lower=0.005 upper=0 effort=1 velocity=1
- added joint wg-front-left-2-joint: type prismatic, parent wh-front-left, child wg-front-left-2, origin xyz=0 0 0 rpy=0 2.51327412287 0, limit lower=0.005 upper=0 effort=1 velocity=1
- added joint wg-front-left-3-joint: type prismatic, parent wh-front-left, child wg-front-left-3, origin xyz=0 0 0 rpy=0 3.76991118431 0, limit lower=0.005 upper=0 effort=1 velocity=1
- added joint wg-front-left-4-joint: type prismatic, parent wh-front-left, child wg-front-left-4, origin xyz=0 0 0 rpy=0 5.02654824574 0, limit lower=0.005 upper=0 effort=1 velocity=1
- added joint wg-front-left-5-joint: type prismatic, parent wh-front-left, child wg-front-left-5, origin xyz=0 0 0 rpy=0 6.28318530718 0, limit lower=0.005 upper=0 effort=1 velocity=1
- added joint wg-front-right-1-joint: type prismatic, parent wh-front-right, child wg-front-right-1, origin xyz=0 0 0 rpy=0 1.25663706144 0, limit lower=0.005 upper=0 effort=1 velocity=1
- added joint wg-front-right-2-joint: type prismatic, parent wh-front-right, child wg-front-right-2, origin xyz=0 0 0 rpy=0 2.51327412287 0, limit lower=0.005 upper=0 effort=1 velocity=1
- added joint wg-front-right-3-joint: type prismatic, parent wh-front-right, child wg-front-right-3, origin xyz=0 0 0 rpy=0 3.76991118431 0, limit lower=0.005 upper=0 effort=1 velocity=1
- added joint wg-front-right-4-joint: type prismatic, parent wh-front-right, child wg-front-right-4, origin xyz=0 0 0 rpy=0 5.02654824574 0, limit lower=0.005 upper=0 effort=1 velocity=1
- added joint wg-front-right-5-joint: type prismatic, parent wh-front-right, child wg-front-right-5, origin xyz=0 0 0 rpy=0 6.28318530718 0, limit lower=0.005 upper=0 effort=1 velocity=1
- joint ax-back-left: origin xyz=-0.05 -0.0375 0.011 rpy=0 0 0  -> xyz=-0.05 -0.0375 0.011 rpy=0 0 0
- joint ax-back-right: origin xyz=-0.05 0.0375 0.011 rpy=0 0 0  -> xyz=-0.05 0.0375 0.011 rpy=0 0 0
- joint ax-front-left: origin xyz=0.05 -0.0375 0.011 rpy=0 0 0  -> xyz=0.05 -0.0375 0.011 rpy=0 0 0
- joint ax-front-right: origin xyz=0.05 0.0375 0.011 rpy=0 0 0  -> xyz=0.05 0.0375 0.011 rpy=0 0 0

File: src/adabot_description/urdf/adabot.xacro (robot description, xacro)
@@ -12,4 +12,8 @@
     <xacro:property name="ch_height" value="0.035" />
     <xacro:property name="ch_mass" value="${500*ch_length*ch_width*ch_height}" />
+    <xacro:property name="wg_length" value="0.002" />
+    <xacro:property name="wg_width" value="0.001" />
+    <xacro:property name="wg_height" value="0.04" />
+    <xacro:property name="wg_mass" value="${500*wg_length*wg_width*wg_height}" />
     <xacro:property name="zoffset" value="${wh_radius*1.1/2}" />
     <!--
@@ -22,4 +26,7 @@
     <material name="white">
         <color rgba="1 1 1 1" />
+    </material>
+    <material name="red">
+        <color rgba=".255, 0, 0, .001" />
     </material>
     <!--
@@ -59,6 +66,51 @@
             <parent link="${parent}" />
             <child link="wh-${suffix}" />
-            <origin rpy="0 0 0 " xyz="${ch_length/2*reflect_fb} ${(wh_length+ch_width)/2*reflect_lr} ${zoffset}" />
+            <origin rpy="0 0 0" xyz="${ch_length/2*reflect_fb} ${(wh_length+ch_width)/2*reflect_lr} ${zoffset}" />
             <axis xyz="${ax_axis}" />
+        </joint>
+        <xacro:weg wheel="${suffix}" number="1" parent="wh-${suffix}" />
+        <xacro:weg wheel="${suffix}" number="2" parent="wh-${suffix}" />
+        <xacro:weg wheel="${suffix}" number="3" parent="wh-${suffix}" />
+        <xacro:weg wheel="${suffix}" number="4" parent="wh-${suffix}" />
+        <xacro:weg wheel="${suffix}" number="5" parent="wh-${suffix}" />
+    </xacro:macro>
+    <!--
+         Macro for creating weg geoms
+    -->
+    <xacro:property name="wg_origin_geom">
+        <origin rpy="0 0 0" xyz="0 0 0" />
+        <geometry>
+            <box size="${wg_length} ${wg_width} ${wg_height}" />
+        </geometry>
+    </xacro:property>
+    <!--
+         Macro for creating wegs
+    -->
+    <xacro:macro name="weg" params="wheel number parent">
+        <link name="wg-${wheel}-${number}">
+            <visual>
+                <xacro:insert_block name="wg_origin_geom" />
+                <material name="white" />
+            </visual>
+            <collision>
+                <xacro:insert_block name="wg_origin_geom" />
+            </collision>
+            <inertial>
+                <mass value="${wg_mass}" />
+                <inertia
+                    ixx="${(1/12)*wg_mass*(wg_width**2 + wg_height**2)}"
+                    ixy="0"
+                    ixz="0"
+                    iyy="${(1/12)*wg_mass*(wg_length**2 + wg_height**2)}"
+                    iyz="0"
+                    izz="${(1/12)*wg_mass*(wg_length**2 + wg_width**2)}"
+                    />
+            </inertial>
+        </link>
+        <joint name="wg-${wheel}-${number}-joint" type="prismatic">
+            <parent link="${parent}" />
+            <child link="wg-${wheel}-${number}" />
+            <origin rpy="0 ${2*pi*(number/5)} 0" xyz="0 0 0" />
+            <limit upper="0" lower="0.005" effort="1" velocity="1" />
         </joint>
     </xacro:macro>

Commit message: Fixed weg dimensions

File: src/adabot_description/urdf/adabot.urdf (robot description, URDF)
Before this commit: robot adabot, 25 links, 24 joints
Links:
- link wg-back-left-1: geometry collision box size=0.04 0.001 0.002; visual box size=0.04 0.001 0.002
- link wg-back-left-2: geometry collision box size=0.04 0.001 0.002; visual box size=0.04 0.001 0.002
- link wg-back-left-3: geometry collision box size=0.04 0.001 0.002; visual box size=0.04 0.001 0.002
- link wg-back-left-4: geometry collision box size=0.04 0.001 0.002; visual box size=0.04 0.001 0.002
- link wg-back-left-5: geometry collision box size=0.04 0.001 0.002; visual box size=0.04 0.001 0.002
- link wg-back-right-1: geometry collision box size=0.04 0.001 0.002; visual box size=0.04 0.001 0.002
- link wg-back-right-2: geometry collision box size=0.04 0.001 0.002; visual box size=0.04 0.001 0.002
- link wg-back-right-3: geometry collision box size=0.04 0.001 0.002; visual box size=0.04 0.001 0.002
- link wg-back-right-4: geometry collision box size=0.04 0.001 0.002; visual box size=0.04 0.001 0.002
- link wg-back-right-5: geometry collision box size=0.04 0.001 0.002; visual box size=0.04 0.001 0.002
- link wg-front-left-1: geometry collision box size=0.04 0.001 0.002; visual box size=0.04 0.001 0.002
- link wg-front-left-2: geometry collision box size=0.04 0.001 0.002; visual box size=0.04 0.001 0.002
- link wg-front-left-3: geometry collision box size=0.04 0.001 0.002; visual box size=0.04 0.001 0.002
- link wg-front-left-4: geometry collision box size=0.04 0.001 0.002; visual box size=0.04 0.001 0.002
- link wg-front-left-5: geometry collision box size=0.04 0.001 0.002; visual box size=0.04 0.001 0.002
- link wg-front-right-1: geometry collision box size=0.04 0.001 0.002; visual box size=0.04 0.001 0.002
- link wg-front-right-2: geometry collision box size=0.04 0.001 0.002; visual box size=0.04 0.001 0.002
- link wg-front-right-3: geometry collision box size=0.04 0.001 0.002; visual box size=0.04 0.001 0.002
- link wg-front-right-4: geometry collision box size=0.04 0.001 0.002; visual box size=0.04 0.001 0.002
- link wg-front-right-5: geometry collision box size=0.04 0.001 0.002; visual box size=0.04 0.001 0.002
Joints:
- joint wg-back-left-1-joint: limit lower=0.005 upper=0 effort=1 velocity=1 -> lower=0 upper=0.008 effort=1 velocity=1
- joint wg-back-left-2-joint: limit lower=0.005 upper=0 effort=1 velocity=1 -> lower=0 upper=0.008 effort=1 velocity=1
- joint wg-back-left-3-joint: limit lower=0.005 upper=0 effort=1 velocity=1 -> lower=0 upper=0.008 effort=1 velocity=1
- joint wg-back-left-4-joint: limit lower=0.005 upper=0 effort=1 velocity=1 -> lower=0 upper=0.008 effort=1 velocity=1
- joint wg-back-left-5-joint: limit lower=0.005 upper=0 effort=1 velocity=1 -> lower=0 upper=0.008 effort=1 velocity=1
- joint wg-back-right-1-joint: limit lower=0.005 upper=0 effort=1 velocity=1 -> lower=0 upper=0.008 effort=1 velocity=1
- joint wg-back-right-2-joint: limit lower=0.005 upper=0 effort=1 velocity=1 -> lower=0 upper=0.008 effort=1 velocity=1
- joint wg-back-right-3-joint: limit lower=0.005 upper=0 effort=1 velocity=1 -> lower=0 upper=0.008 effort=1 velocity=1
- joint wg-back-right-4-joint: limit lower=0.005 upper=0 effort=1 velocity=1 -> lower=0 upper=0.008 effort=1 velocity=1
- joint wg-back-right-5-joint: limit lower=0.005 upper=0 effort=1 velocity=1 -> lower=0 upper=0.008 effort=1 velocity=1
- joint wg-front-left-1-joint: limit lower=0.005 upper=0 effort=1 velocity=1 -> lower=0 upper=0.008 effort=1 velocity=1
- joint wg-front-left-2-joint: limit lower=0.005 upper=0 effort=1 velocity=1 -> lower=0 upper=0.008 effort=1 velocity=1
- joint wg-front-left-3-joint: limit lower=0.005 upper=0 effort=1 velocity=1 -> lower=0 upper=0.008 effort=1 velocity=1
- joint wg-front-left-4-joint: limit lower=0.005 upper=0 effort=1 velocity=1 -> lower=0 upper=0.008 effort=1 velocity=1
- joint wg-front-left-5-joint: limit lower=0.005 upper=0 effort=1 velocity=1 -> lower=0 upper=0.008 effort=1 velocity=1
- joint wg-front-right-1-joint: limit lower=0.005 upper=0 effort=1 velocity=1 -> lower=0 upper=0.008 effort=1 velocity=1
- joint wg-front-right-2-joint: limit lower=0.005 upper=0 effort=1 velocity=1 -> lower=0 upper=0.008 effort=1 velocity=1
- joint wg-front-right-3-joint: limit lower=0.005 upper=0 effort=1 velocity=1 -> lower=0 upper=0.008 effort=1 velocity=1
- joint wg-front-right-4-joint: limit lower=0.005 upper=0 effort=1 velocity=1 -> lower=0 upper=0.008 effort=1 velocity=1
- joint wg-front-right-5-joint: limit lower=0.005 upper=0 effort=1 velocity=1 -> lower=0 upper=0.008 effort=1 velocity=1

File: src/adabot_description/urdf/adabot.xacro (robot description, xacro)
@@ -12,7 +12,7 @@
     <xacro:property name="ch_height" value="0.035" />
     <xacro:property name="ch_mass" value="${500*ch_length*ch_width*ch_height}" />
-    <xacro:property name="wg_length" value="0.002" />
+    <xacro:property name="wg_length" value="${wh_radius*2}" />
     <xacro:property name="wg_width" value="0.001" />
-    <xacro:property name="wg_height" value="0.04" />
+    <xacro:property name="wg_height" value="0.002" />
     <xacro:property name="wg_mass" value="${500*wg_length*wg_width*wg_height}" />
     <xacro:property name="zoffset" value="${wh_radius*1.1/2}" />
@@ -112,5 +112,5 @@
             <child link="wg-${wheel}-${number}" />
             <origin rpy="0 ${2*pi*(number/5)} 0" xyz="0 0 0" />
-            <limit upper="0" lower="0.005" effort="1" velocity="1" />
+            <limit upper="${wg_length*.2}" lower="0" effort="1" velocity="1" />
         </joint>
     </xacro:macro>
