Commit message: Updated and reorganized the xacro files.

File: adabot_description/urdf/adabot.base.xacro (robot description, xacro)
@@ -2,36 +2,86 @@
 <robot xmlns:xacro="http://www.ros.org/wiki/xacro" name="adabot">
     <!--
-         Properties for the geometries
+         Properties for the robot bodies
     -->
+    <xacro:property name="PI" value="3.1415926535897931"/>
+    <!-- Typical density of plastics -->
+    <xacro:property name="mat_density" value="1000.0" />
+    <!-- Wheel parameters -->
     <xacro:property name="wh_radius" value="0.02" />
     <xacro:property name="wh_length" value="0.005" />
-    <xacro:property name="wh_mass" value="${500*3.145927*(wh_radius**2)*wh_length}" />
+    <xacro:property name="wh_mass" value="${mat_density*PI*(wh_radius**2)*wh_length}" />
+    <!-- Axle parameters -->
     <xacro:property name="ax_axis" value="0 1 0" />
+    <!-- Chassis parameters -->
     <xacro:property name="ch_length" value="0.1" />
     <xacro:property name="ch_width" value="0.07" />
     <xacro:property name="ch_height" value="0.035" />
-    <xacro:property name="ch_mass" value="${500*ch_length*ch_width*ch_height}" />
+    <xacro:property name="ch_mass" value="${mat_density*ch_length*ch_width*ch_height}" />
+    <!-- Weg parameters -->
     <xacro:property name="wg_length" value="${wh_radius*2}" />
     <xacro:property name="wg_width" value="0.001" />
     <xacro:property name="wg_height" value="0.002" />
-    <xacro:property name="wg_mass" value="${500*wg_length*wg_width*wg_height}" />
+    <xacro:property name="wg_mass" value="${mat_density*wg_length*wg_width*wg_height}" />
+    <!-- Vertical offset so that the robot starts above ground -->
     <xacro:property name="zoffset" value="${wh_radius*1.1/2}" />
     <!--
-         Properties for names and colors
+         Properties for names, colors, and Gazebo
     -->
+    <!-- The chassis is the parent of several other links, so we need it's name -->
     <xacro:property name="chassisname" value="base_link" />
-    <material name="black">
-        <color rgba="0 0 0 1" />
-    </material>
-    <material name="white">
-        <color rgba="1 1 1 1" />
-    </material>
-    <material name="red">
-        <color rgba=".255, 0, 0, .001" />
-    </material>
+    <!-- Import colors defined for Rviz -->
+    <xacro:include filename="$(find adabot_description)/urdf/adabot.materials.xacro" />
+    <!-- Import tags needed by Gazebo -->
+    <xacro:include filename="$(find adabot_description)/urdf/adabot.gazebo.xacro" />
+    <!--
+         Macro for creating weg geoms
+    -->
+    <xacro:property name="wg_origin_geom">
+        <origin rpy="0 0 0" xyz="0 0 0" />
+        <geometry>
+            <box size="${wg_length} ${wg_width} ${wg_height}" />
+        </geometry>
+    </xacro:property>
+    <!--
+         Macro for creating wegs
+            wheel  : the suffix of the parent wheel
+            number : a unique identifier for each weg
+            parent : the full name of the parent link
+            total  : the number of wegs (used to calculate angles)
+    -->
+    <xacro:macro name="weg" params="wheel number parent total">
+        <xacro:property name="wg_name" value="wg-${wheel}-${number}" />
+        <link name="${wg_name}">
+            <visual>
+                <xacro:insert_block name="wg_origin_geom" />
+                <material name="white" />
+            </visual>
+            <collision>
+                <xacro:insert_block name="wg_origin_geom" />
+            </collision>
+            <inertial>
+                <mass value="${wg_mass}" />
+                <inertia
+                    ixx="${(1/12)*wg_mass*(wg_width**2 + wg_height**2)}"
+                    ixy="0"
+                    ixz="0"
+                    iyy="${(1/12)*wg_mass*(wg_length**2 + wg_height**2)}"
+                    iyz="0"
+                    izz="${(1/12)*wg_mass*(wg_length**2 + wg_width**2)}"
+                    />
+            </inertial>
+        </link>
+        <joint name="${wg_name}-joint" type="prismatic">
+            <parent link="${parent}" />
+            <child link="${wg_name}" />
+            <origin rpy="0 ${2*PI*(number/total)} 0" xyz="0 0 0" />
+            <limit upper="${wg_length*.2}" lower="0" effort="1" velocity="1" />
+        </joint>
+    </xacro:macro>
     <!--
          Macro for creating wheel geoms
     -->
     <xacro:property name="wh_orig_geom">
+        <!-- Cylinders default with their height along the z axis -->
         <origin rpy="1.57075 0 0" xyz="0 0 0" />
         <geometry>
@@ -41,7 +91,12 @@
     <!--
          Macro for creating wheels
+            reflect_lr : is the wheel left (-1) or right (1)
+            reflect_fb : is the wheel front (1) or back (-1)
+            suffix     : give the wheel a unique name
+            parent     : to what link is this wheel attached
     -->
     <xacro:macro name="wheel" params="reflect_lr reflect_fb suffix parent">
-        <link name="wh-${suffix}">
+        <xacro:property name="wh_name" value="wh-${suffix}" />
+        <link name="${wh_name}">
             <visual>
                 <xacro:insert_block name="wh_orig_geom" />
@@ -65,53 +120,20 @@
         <joint name="ax-${suffix}" type="continuous">
             <parent link="${parent}" />
-            <child link="wh-${suffix}" />
+            <child link="${wh_name}" />
             <origin rpy="0 0 0" xyz="${ch_length/2*reflect_fb} ${(wh_length+ch_width)/2*reflect_lr} ${zoffset}" />
             <axis xyz="${ax_axis}" />
         </joint>
-        <xacro:weg wheel="${suffix}" number="1" parent="wh-${suffix}" />
-        <xacro:weg wheel="${suffix}" number="2" parent="wh-${suffix}" />
-        <xacro:weg wheel="${suffix}" number="3" parent="wh-${suffix}" />
-        <xacro:weg wheel="${suffix}" number="4" parent="wh-${suffix}" />
-        <xacro:weg wheel="${suffix}" number="5" parent="wh-${suffix}" />
-    </xacro:macro>
-    <!--
-         Macro for creating weg geoms
-    -->
-    <xacro:property name="wg_origin_geom">
-        <origin rpy="0 0 0" xyz="0 0 0" />
-        <geometry>
-            <box size="${wg_length} ${wg_width} ${wg_height}" />
-        </geometry>
-    </xacro:property>
-    <!--
-         Macro for creating wegs
-    -->
-    <xacro:macro name="weg" params="wheel number parent">
-        <link name="wg-${wheel}-${number}">
-            <visual>
-                <xacro:insert_block name="wg_origin_geom" />
-                <material name="white" />
-            </visual>
-            <collision>
-                <xacro:insert_block name="wg_origin_geom" />
-            </collision>
-            <inertial>
-                <mass value="${wg_mass}" />
-                <inertia
-                    ixx="${(1/12)*wg_mass*(wg_width**2 + wg_height**2)}"
-                    ixy="0"
-                    ixz="0"
-                    iyy="${(1/12)*wg_mass*(wg_length**2 + wg_height**2)}"
-                    iyz="0"
-                    izz="${(1/12)*wg_mass*(wg_length**2 + wg_width**2)}"
-                    />
-            </inertial>
-        </link>
-        <joint name="wg-${wheel}-${number}-joint" type="prismatic">
-            <parent link="${parent}" />
-            <child link="wg-${wheel}-${number}" />
-            <origin rpy="0 ${2*pi*(number/5)} 0" xyz="0 0 0" />
-            <limit upper="${wg_length*.2}" lower="0" effort="1" velocity="1" />
-        </joint>
+        <!-- http://answers.ros.org/question/38956/pass-parameters-to-xacro-in-launch-file/
+                (1) add a parameter to the launch files
+                (2) pass the parameter to xacro.py (the above link)
+                (3) set a default value in this file
+                (4) pass the value to the wheel macro
+                (5) have some ugly conditionals below
+        -->
+        <xacro:weg wheel="${suffix}" number="1" parent="${wh_name}" />
+        <xacro:weg wheel="${suffix}" number="2" parent="${wh_name}" />
+        <xacro:weg wheel="${suffix}" number="3" parent="${wh_name}" />
+        <xacro:weg wheel="${suffix}" number="4" parent="${wh_name}" />
+        <xacro:weg wheel="${suffix}" number="5" parent="${wh_name}" />
     </xacro:macro>
     <!--
