Commit message: Working on a jitter problem.

File: adabot_description/urdf/adabot.parameters.xacro (robot description, xacro)
@@ -16,5 +16,5 @@
     <xacro:property name="ch_mass"    value="${ch_density * ch_length * ch_width * ch_height}" />
     <!-- Wheel parameters -->
-    <xacro:property name="wh_density_factor" value="0.4" />
+    <xacro:property name="wh_density_factor" value="0.1" />
     <xacro:property name="wh_density" value="${mat_density * wh_density_factor}" />
     <xacro:property name="wh_radius"  value="${0.020 * SCALE}" />
@@ -22,9 +22,9 @@
     <xacro:property name="wh_mass"    value="${wh_density * PI * (wh_radius**2) * wh_length}" />
     <!-- Weg parameters -->
-    <xacro:property name="wg_length" value="${wh_radius}" />
+    <xacro:property name="wg_length" value="${wh_radius * 0.75}" />
     <xacro:property name="wg_width"  value="${0.001 * SCALE}" />
     <xacro:property name="wg_height" value="${0.002 * SCALE}" />
     <xacro:property name="wg_mass"   value="${mat_density * wg_length * wg_width * wg_height}" />
     <!-- Vertical offset so that the robot starts above ground -->
-    <xacro:property name="z_offset" value="${wh_radius * 10}" />
+    <xacro:property name="z_offset" value="${wh_radius * 2}" />
 </robot>

Commit message: Moved rockySurface to correct directory.

File: adabot_description/urdf/adabot.parameters.xacro (robot description, xacro)
@@ -22,5 +22,5 @@
     <xacro:property name="ch_density_factor" value="0.4" />
     <xacro:property name="ch_density" value="${mat_density * ch_density_factor}" />
-    <xacro:property name="ch_length"  value="${0.100 * 0.65 * $(arg ch_length_factor) * SCALE}" />
+    <xacro:property name="ch_length"  value="${0.100 * $(arg ch_length_factor) * SCALE}" />
     <xacro:property name="ch_width"   value="${0.070 * $(arg ch_width_factor) * SCALE}" />
     <xacro:property name="ch_height"  value="${0.025 * SCALE}" />
