Commit message: Merged my velocity controller branch with master.

File: adabot_description/urdf/adabot.macros.xacro (robot description, xacro)
@@ -23,6 +23,9 @@
     -->
     <xacro:macro name="wheel" params="reflect_lr reflect_fr suffix">
+        <!-- The name of the current wheel -->
         <xacro:property name="wheel_name" value="${suffix}_wheel" />
+        <!-- Add the wheel's Gazebo material -->
         <xacro:gz_wheel_material name="${wheel_name}" />
+        <!-- The wheel's rigid body -->
         <link name="${wheel_name}">
             <visual>
@@ -46,4 +49,5 @@
             </inertial>
         </link>
+        <!-- Connect the wheel to the chassis -->
         <joint name="${wheel_name}_joint" type="continuous">
             <parent link="chassis" />
@@ -53,4 +57,9 @@
             <limit effort="10" velocity="100" />
         </joint>
+        <!--
+             Attach a velocity controller to the wheel's joint
+                Any changes to the wheel joint's name will need to be reflected
+                  in 'adabot.control.yaml' and 'adabot.control.launch'.
+        -->
         <transmission name="${wheel_name}_transmission" type="SimpleTransmission">
             <type>transmission_interface/SimpleTransmission</type>
@@ -63,4 +72,56 @@
             </actuator>
         </transmission>
+        <!-- Add wegs to this wheel -->
+        <xacro:weg wheel="${suffix}" number="1" parent="${wh_name}" total="5" />
+        <xacro:weg wheel="${suffix}" number="2" parent="${wh_name}" total="5" />
+        <xacro:weg wheel="${suffix}" number="3" parent="${wh_name}" total="5" />
+        <xacro:weg wheel="${suffix}" number="4" parent="${wh_name}" total="5" />
+        <xacro:weg wheel="${suffix}" number="5" parent="${wh_name}" total="5" />
+    </xacro:macro>
+    <!-- Create the weg geometry (for visuals and collisions) -->
+    <xacro:property name="wg_origin_geom">
+        <origin rpy="0 0 0" xyz="0 0 0" />
+        <geometry>
+            <box size="${wg_length} ${wg_width} ${wg_height}" />
+        </geometry>
+    </xacro:property>
+    <!--
+         Macro for creating wegs
+            wheel  : the suffix of the parent wheel
+            number : a unique identifier for each weg
+            parent : the full name of the parent link
+            total  : the number of wegs (used to calculate angles)
+    -->
+    <xacro:macro name="weg" params="wheel number parent total">
+        <!-- The name of the current weg (based on the parent wheel's name) -->
+        <xacro:property name="wg_name" value="wg_${wheel}_${number}" />
+        <!-- The weg's rigid body -->
+        <link name="${wg_name}">
+            <visual>
+                <xacro:insert_block name="wg_origin_geom" />
+                <material name="white" />
+            </visual>
+            <collision>
+                <xacro:insert_block name="wg_origin_geom" />
+            </collision>
+            <inertial>
+                <mass value="${wg_mass}" />
+                <inertia
+                    ixx="${(1/12)*wg_mass*(wg_width**2 + wg_height**2)}"
+                    ixy="0"
+                    ixz="0"
+                    iyy="${(1/12)*wg_mass*(wg_length**2 + wg_height**2)}"
+                    iyz="0"
+                    izz="${(1/12)*wg_mass*(wg_length**2 + wg_width**2)}"
+                    />
+            </inertial>
+        </link>
+        <!-- Connect the weg to the wheel with a prismatic joint -->
+        <joint name="${wg_name}_joint" type="prismatic">
+            <parent link="${parent}" />
+            <child link="${wg_name}" />
+            <origin rpy="0 ${2*PI*(number/total)} 0" xyz="0 0 0" />
+            <limit upper="${wg_length*.2}" lower="0" effort="1" velocity="1" />
+        </joint>
     </xacro:macro>
 </robot>

File: adabot_description/urdf/adabot.parameters.xacro (robot description, xacro)
@@ -1,5 +1,5 @@
 <?xml version="1.0"?>
 <robot xmlns:xacro="http://www.ros.org/wiki/xacro" name="adabot">
-     <!--
+    <!--
          Properties for the robot bodies
     -->
@@ -21,4 +21,9 @@
     <xacro:property name="wh_length"  value="${0.005 * SCALE}" />
     <xacro:property name="wh_mass"    value="${wh_density * PI * (wh_radius**2) * wh_length}" />
+    <!-- Weg parameters -->
+    <xacro:property name="wg_length" value="${wh_radius*2}" />
+    <xacro:property name="wg_width"  value="${0.001 * SCALE}" />
+    <xacro:property name="wg_height" value="${0.002 * SCALE}" />
+    <xacro:property name="wg_mass"   value="${mat_density * wg_length * wg_width * wg_height}" />
     <!-- Vertical offset so that the robot starts above ground -->
     <xacro:property name="z_offset" value="${wh_radius * 10}" />

Commit message: Adding linear servos to the wegs.

File: adabot_description/urdf/adabot.macros.xacro (robot description, xacro)
@@ -55,8 +55,8 @@
             <origin xyz="${ch_length/2*reflect_fr} ${(wh_length+ch_width)/2*reflect_lr} 0" rpy="0 0 0" />
             <axis xyz="0 1 0" />
-            <limit effort="10" velocity="100" />
+            <limit effort="10" velocity="10" />
         </joint>
         <!--
-             Attach a velocity controller to the wheel's joint
+             Attach a VELOCITY controller to the wheel's joint
                 Any changes to the wheel joint's name will need to be reflected
                   in 'adabot.control.yaml' and 'adabot.control.launch'.
@@ -73,13 +73,13 @@
         </transmission>
         <!-- Add wegs to this wheel -->
-        <xacro:weg wheel="${suffix}" number="1" parent="${wh_name}" total="5" />
-        <xacro:weg wheel="${suffix}" number="2" parent="${wh_name}" total="5" />
-        <xacro:weg wheel="${suffix}" number="3" parent="${wh_name}" total="5" />
-        <xacro:weg wheel="${suffix}" number="4" parent="${wh_name}" total="5" />
-        <xacro:weg wheel="${suffix}" number="5" parent="${wh_name}" total="5" />
+        <xacro:weg wheel="${suffix}" number="1" parent="${wheel_name}" total="5" />
+        <xacro:weg wheel="${suffix}" number="2" parent="${wheel_name}" total="5" />
+        <xacro:weg wheel="${suffix}" number="3" parent="${wheel_name}" total="5" />
+        <xacro:weg wheel="${suffix}" number="4" parent="${wheel_name}" total="5" />
+        <xacro:weg wheel="${suffix}" number="5" parent="${wheel_name}" total="5" />
     </xacro:macro>
     <!-- Create the weg geometry (for visuals and collisions) -->
     <xacro:property name="wg_origin_geom">
-        <origin rpy="0 0 0" xyz="0 0 0" />
+        <origin xyz="${wh_radius/2} 0 0" rpy="0 0 0" />
         <geometry>
             <box size="${wg_length} ${wg_width} ${wg_height}" />
@@ -95,7 +95,7 @@
     <xacro:macro name="weg" params="wheel number parent total">
         <!-- The name of the current weg (based on the parent wheel's name) -->
-        <xacro:property name="wg_name" value="wg_${wheel}_${number}" />
+        <xacro:property name="weg_name" value="${wheel}_weg_${number}" />
         <!-- The weg's rigid body -->
-        <link name="${wg_name}">
+        <link name="${weg_name}">
             <visual>
                 <xacro:insert_block name="wg_origin_geom" />
@@ -118,10 +118,29 @@
         </link>
         <!-- Connect the weg to the wheel with a prismatic joint -->
-        <joint name="${wg_name}_joint" type="prismatic">
+        <joint name="${weg_name}_joint" type="prismatic">
             <parent link="${parent}" />
-            <child link="${wg_name}" />
-            <origin rpy="0 ${2*PI*(number/total)} 0" xyz="0 0 0" />
-            <limit upper="${wg_length*.2}" lower="0" effort="1" velocity="1" />
+            <child link="${weg_name}" />
+            <origin xyz="0 0 0" rpy="0 ${2 * PI * (number/total)} 0" />
+            <limit upper="${wh_radius * 0.7}" lower="0" effort="10" velocity="10" />
         </joint>
+        <!--
+             Attach a POSITION controller to each weg prismatic joint
+                Any changes to the wheel joint's name will need to be reflected
+                  in 'adabot.control.yaml' and 'adabot.control.launch'.
+                Also note that, technically, all wegs for a single joint should be
+                  controlled together (a single transimission for each weg set).
+                  However, I do not think this will be possible given that the transmission
+                  interface requires a single process value for each motor.
+        -->
+        <transmission name="${weg_name}_transmission" type="SimpleTransmission">
+            <type>transmission_interface/SimpleTransmission</type>
+            <joint name="${weg_name}_joint">
+                <hardwareInterface>hardware_interface/EffortJointInterface</hardwareInterface>
+            </joint>
+            <actuator name="${weg_name}_motor">
+                <hardwareInterface>hardware_interface/EffortJointInterface</hardwareInterface>
+                <mechanicalReduction>1</mechanicalReduction>
+            </actuator>
+        </transmission>
     </xacro:macro>
 </robot>

File: adabot_description/urdf/adabot.main.xacro (robot description, xacro)
@@ -36,5 +36,5 @@
         <child link="chassis" />
     </joint>
-    <!-- Add the wheels -->
+    <!-- Add the wheels (note, wegs are created with the wheels) -->
     <xacro:wheel reflect_lr="1"  reflect_fr="1"  suffix="front_left"  />
     <xacro:wheel reflect_lr="-1" reflect_fr="1"  suffix="front_right" />

File: adabot_description/urdf/adabot.parameters.xacro (robot description, xacro)
@@ -22,5 +22,5 @@
     <xacro:property name="wh_mass"    value="${wh_density * PI * (wh_radius**2) * wh_length}" />
     <!-- Weg parameters -->
-    <xacro:property name="wg_length" value="${wh_radius*2}" />
+    <xacro:property name="wg_length" value="${wh_radius}" />
     <xacro:property name="wg_width"  value="${0.001 * SCALE}" />
     <xacro:property name="wg_height" value="${0.002 * SCALE}" />

Commit message: Fixed the wegs to eliminate jitter (for testing), added sphereical weg tips, and changed the wheels from cylinders to sphere.

File: adabot_description/urdf/adabot.macros.xacro (robot description, xacro)
@@ -9,9 +9,18 @@
     </xacro:property>
     <!-- Create the wheel geometry (for visuals and collisions) -->
+    <!-- <xacro:property name="wheel_geometry"> -->
+        <!-- Cylinders default with their height along the z axis -->
+<!--         <origin xyz="0 0 0" rpy="${PI/2} 0 0" />
+        <geometry>
+            <cylinder length="${wh_length}" radius="${wh_radius}" />
+        </geometry>
+    </xacro:property>
+ -->
     <xacro:property name="wheel_geometry">
         <!-- Cylinders default with their height along the z axis -->
         <origin xyz="0 0 0" rpy="${PI/2} 0 0" />
         <geometry>
-            <cylinder length="${wh_length}" radius="${wh_radius}" />
+            <!-- <cylinder length="${wh_length}" radius="${wh_radius}" /> -->
+            <sphere radius="${wh_radius}" />
         </geometry>
     </xacro:property>
@@ -80,8 +89,21 @@
     </xacro:macro>
     <!-- Create the weg geometry (for visuals and collisions) -->
-    <xacro:property name="wg_origin_geom">
+<!--     <xacro:property name="weg_geometry">
         <origin xyz="${wh_radius/2} 0 0" rpy="0 0 0" />
         <geometry>
             <box size="${wg_length} ${wg_width} ${wg_height}" />
+        </geometry>
+    </xacro:property> -->
+    <xacro:property name="weg_geometry">
+        <origin xyz="${wh_radius} 0 0" rpy="0 0 0" />
+        <geometry>
+            <box size="${wg_length} ${wg_width} ${wg_height}" />
+        </geometry>
+    </xacro:property>
+    <!-- Create a geometry for the weg tip -->
+    <xacro:property name="weg_tip_geometry">
+        <!-- <origin xyz="${wh_radius} 0 0" rpy="0 0 0" /> -->
+        <geometry>
+            <sphere radius="${wt_radius}" />
         </geometry>
     </xacro:property>
@@ -99,9 +121,9 @@
         <link name="${weg_name}">
             <visual>
-                <xacro:insert_block name="wg_origin_geom" />
+                <xacro:insert_block name="weg_geometry" />
                 <material name="white" />
             </visual>
             <collision>
-                <xacro:insert_block name="wg_origin_geom" />
+                <xacro:insert_block name="weg_geometry" />
             </collision>
             <inertial>
@@ -118,9 +140,15 @@
         </link>
         <!-- Connect the weg to the wheel with a prismatic joint -->
-        <joint name="${weg_name}_joint" type="prismatic">
+<!--         <joint name="${weg_name}_joint" type="prismatic">
             <parent link="${parent}" />
             <child link="${weg_name}" />
             <origin xyz="0 0 0" rpy="0 ${2 * PI * (number/total)} 0" />
             <limit upper="${wh_radius * 0.7}" lower="0" effort="10" velocity="10" />
+        </joint> -->
+        <joint name="${weg_name}_joint" type="fixed">
+            <parent link="${parent}" />
+            <child link="${weg_name}" />
+            <origin xyz="0 0 0" rpy="0 ${2 * PI * (number/total)} 0" />
+            <!-- <limit upper="${wh_radius * 0.7}" lower="0" effort="10" velocity="10" /> -->
         </joint>
         <!--
@@ -133,5 +161,5 @@
                   interface requires a single process value for each motor.
         -->
-        <transmission name="${weg_name}_transmission" type="SimpleTransmission">
+<!--         <transmission name="${weg_name}_transmission" type="SimpleTransmission">
             <type>transmission_interface/SimpleTransmission</type>
             <joint name="${weg_name}_joint">
@@ -142,5 +170,34 @@
                 <mechanicalReduction>1</mechanicalReduction>
             </actuator>
-        </transmission>
+        </transmission> -->
+        <!-- Attach a sphere to the end of the weg for better physics (less jitter) -->
+        <link name="${weg_name}_tip">
+            <visual>
+                <xacro:insert_block name="weg_tip_geometry" />
+                <material name="black" />
+            </visual>
+            <collision>
+                <xacro:insert_block name="weg_tip_geometry" />
+            </collision>
+            <inertial>
+                <mass value="${wt_mass}" />
+                <inertia
+                    ixx="${(2/5) * wt_mass * wt_radius * wt_radius}"
+                    ixy="0"
+                    ixz="0"
+                    iyy="${(2/5) * wt_mass * wt_radius * wt_radius}"
+                    iyz="0"
+                    izz="${(2/5) * wt_mass * wt_radius * wt_radius}"
+                    />
+            </inertial>
+        </link>
+        <!-- Connect the weg tip to the weg -->
+        <joint name="${weg_name}_tip_joint" type="fixed">
+            <parent link="${weg_name}" />
+            <child link="${weg_name}_tip" />
+            <origin xyz="${wg_length/2 + wh_radius} 0 0" rpy="0 0 0" />
+            <!-- <origin xyz="0 0 0" rpy="0 ${2 * PI * (number/total)} 0" /> -->
+            <!-- <limit upper="${wh_radius * 0.7}" lower="0" effort="10" velocity="10" /> -->
+        </joint>
     </xacro:macro>
 </robot>

File: adabot_description/urdf/adabot.parameters.xacro (robot description, xacro)
@@ -22,8 +22,15 @@
     <xacro:property name="wh_mass"    value="${wh_density * PI * (wh_radius**2) * wh_length}" />
     <!-- Weg parameters -->
-    <xacro:property name="wg_length" value="${wh_radius * 0.75}" />
-    <xacro:property name="wg_width"  value="${0.001 * SCALE}" />
-    <xacro:property name="wg_height" value="${0.002 * SCALE}" />
-    <xacro:property name="wg_mass"   value="${mat_density * wg_length * wg_width * wg_height}" />
+    <xacro:property name="wg_density_factor" value="0.5" />
+    <xacro:property name="wg_density" value="${mat_density * wg_density_factor}" />
+    <xacro:property name="wg_length"  value="${wh_radius * 0.75}" />
+    <xacro:property name="wg_width"   value="${0.001 * SCALE}" />
+    <xacro:property name="wg_height"  value="${0.002 * SCALE}" />
+    <xacro:property name="wg_mass"    value="${wg_density * wg_length * wg_width * wg_height}" />
+    <!-- Weg tip parameters -->
+    <xacro:property name="wt_density_factor" value="0.5" />
+    <xacro:property name="wt_density" value="${mat_density * wt_density_factor}" />
+    <xacro:property name="wt_radius"  value="${wg_height * 2}" />
+    <xacro:property name="wt_mass"    value="${wt_density * (4/3) * PI * wt_radius * wt_radius * wt_radius}" />
     <!-- Vertical offset so that the robot starts above ground -->
     <xacro:property name="z_offset" value="${wh_radius * 2}" />

Commit message: I have unlocked the weg prismatic joints. Now I need to test the transmissions again.

File: adabot_description/urdf/adabot.macros.xacro (robot description, xacro)
@@ -9,12 +9,4 @@
     </xacro:property>
     <!-- Create the wheel geometry (for visuals and collisions) -->
-    <!-- <xacro:property name="wheel_geometry"> -->
-        <!-- Cylinders default with their height along the z axis -->
-<!--         <origin xyz="0 0 0" rpy="${PI/2} 0 0" />
-        <geometry>
-            <cylinder length="${wh_length}" radius="${wh_radius}" />
-        </geometry>
-    </xacro:property>
- -->
     <xacro:property name="wheel_geometry">
         <!-- Cylinders default with their height along the z axis -->
@@ -89,12 +81,7 @@
     </xacro:macro>
     <!-- Create the weg geometry (for visuals and collisions) -->
-<!--     <xacro:property name="weg_geometry">
+    <xacro:property name="weg_geometry">
         <origin xyz="${wh_radius/2} 0 0" rpy="0 0 0" />
-        <geometry>
-            <box size="${wg_length} ${wg_width} ${wg_height}" />
-        </geometry>
-    </xacro:property> -->
-    <xacro:property name="weg_geometry">
-        <origin xyz="${wh_radius} 0 0" rpy="0 0 0" />
+        <!-- <origin xyz="${wh_radius} 0 0" rpy="0 0 0" /> -->
         <geometry>
             <box size="${wg_length} ${wg_width} ${wg_height}" />
@@ -140,15 +127,10 @@
         </link>
         <!-- Connect the weg to the wheel with a prismatic joint -->
-<!--         <joint name="${weg_name}_joint" type="prismatic">
+        <joint name="${weg_name}_joint" type="prismatic">
+        <!-- <joint name="${weg_name}_joint" type="fixed"> -->
             <parent link="${parent}" />
             <child link="${weg_name}" />
             <origin xyz="0 0 0" rpy="0 ${2 * PI * (number/total)} 0" />
             <limit upper="${wh_radius * 0.7}" lower="0" effort="10" velocity="10" />
-        </joint> -->
-        <joint name="${weg_name}_joint" type="fixed">
-            <parent link="${parent}" />
-            <child link="${weg_name}" />
-            <origin xyz="0 0 0" rpy="0 ${2 * PI * (number/total)} 0" />
-            <!-- <limit upper="${wh_radius * 0.7}" lower="0" effort="10" velocity="10" /> -->
         </joint>
         <!--
@@ -196,7 +178,7 @@
             <parent link="${weg_name}" />
             <child link="${weg_name}_tip" />
-            <origin xyz="${wg_length/2 + wh_radius} 0 0" rpy="0 0 0" />
-            <!-- <origin xyz="0 0 0" rpy="0 ${2 * PI * (number/total)} 0" /> -->
-            <!-- <limit upper="${wh_radius * 0.7}" lower="0" effort="10" velocity="10" /> -->
+            <!-- The 0.95 is a fudge factor so that weg tips are not aligned with the
+                 wheel radius when commanded to zero. -->
+            <origin xyz="${wh_radius * 0.95 - wt_radius} 0 0" rpy="0 0 0" />
         </joint>
     </xacro:macro>
