Commit message: Code taken from @KeithCissell to partially complete issue #11 (still need to generate control files.

File: adabot_description/urdf/adabot.macros.xacro (robot description, xacro)
@@ -76,9 +76,31 @@
         </transmission>
         <!-- Add wegs to this wheel -->
-        <xacro:weg wheel="${suffix}" number="1" parent="${wheel_name}" total="5" />
-        <xacro:weg wheel="${suffix}" number="2" parent="${wheel_name}" total="5" />
-        <xacro:weg wheel="${suffix}" number="3" parent="${wheel_name}" total="5" />
-        <xacro:weg wheel="${suffix}" number="4" parent="${wheel_name}" total="5" />
-        <xacro:weg wheel="${suffix}" number="5" parent="${wheel_name}" total="5" />
+        <xacro:if value="${wg_per_wheel > 0}">
+            <xacro:weg wheel="${suffix}" number="1" parent="${wheel_name}" total="${wg_per_wheel}" />
+        </xacro:if>
+        <xacro:if value="${wg_per_wheel > 1}">
+            <xacro:weg wheel="${suffix}" number="2" parent="${wheel_name}" total="${wg_per_wheel}" />
+        </xacro:if>
+        <xacro:if value="${wg_per_wheel > 2}">
+            <xacro:weg wheel="${suffix}" number="3" parent="${wheel_name}" total="${wg_per_wheel}" />
+        </xacro:if>
+        <xacro:if value="${wg_per_wheel > 3}">
+            <xacro:weg wheel="${suffix}" number="4" parent="${wheel_name}" total="${wg_per_wheel}" />
+        </xacro:if>
+        <xacro:if value="${wg_per_wheel > 4}">
+            <xacro:weg wheel="${suffix}" number="5" parent="${wheel_name}" total="${wg_per_wheel}" />
+        </xacro:if>
+        <xacro:if value="${wg_per_wheel > 5}">
+            <xacro:weg wheel="${suffix}" number="6" parent="${wheel_name}" total="${wg_per_wheel}" />
+        </xacro:if>
+        <xacro:if value="${wg_per_wheel > 6}">
+            <xacro:weg wheel="${suffix}" number="7" parent="${wheel_name}" total="${wg_per_wheel}" />
+        </xacro:if>
+        <xacro:if value="${wg_per_wheel > 7}">
+            <xacro:weg wheel="${suffix}" number="8" parent="${wheel_name}" total="${wg_per_wheel}" />
+        </xacro:if>
+        <xacro:if value="${wg_per_wheel > 8}">
+            <xacro:weg wheel="${suffix}" number="9" parent="${wheel_name}" total="${wg_per_wheel}" />
+        </xacro:if>
     </xacro:macro>
     <!-- Create the weg geometry (for visuals and collisions) -->

File: adabot_description/urdf/adabot.parameters.xacro (robot description, xacro)
@@ -1,9 +1,17 @@
 <?xml version="1.0"?>
 <robot xmlns:xacro="http://www.ros.org/wiki/xacro" name="adabot">
+    <!--
+         Command line arguments for the adabot
+    -->
+    <xacro:arg name="ch_length"    default="0.100 * 0.65" />
+    <xacro:arg name="ch_width"     default="0.070" />
+    <xacro:arg name="wg_per_wheel" default="5" />
+    <xacro:arg name="wh_radius"    default="0.020" />
+    <xacro:arg name="scale"        default="4" />
     <!--
          Properties for the robot bodies
     -->
     <xacro:property name="PI" value="3.1415926535897931 " />
-    <xacro:property name="SCALE" value="4" />
+    <xacro:property name="SCALE" value="$(arg scale)" />
     <!-- Typical density of plastics -->
     <xacro:property name="mat_density" value="1000.0" />
@@ -11,6 +19,6 @@
     <xacro:property name="ch_density_factor" value="0.4" />
     <xacro:property name="ch_density" value="${mat_density * ch_density_factor}" />
-    <xacro:property name="ch_length"  value="${0.100 * SCALE * 0.65}" />
-    <xacro:property name="ch_width"   value="${0.070 * SCALE}" />
+    <xacro:property name="ch_length"  value="${$(arg ch_length) * SCALE}" />
+    <xacro:property name="ch_width"   value="${$(arg ch_width) * SCALE}" />
     <xacro:property name="ch_height"  value="${0.025 * SCALE}" />
     <xacro:property name="ch_mass"    value="${ch_density * ch_length * ch_width * ch_height}" />
@@ -18,14 +26,15 @@
     <xacro:property name="wh_density_factor" value="0.1" />
     <xacro:property name="wh_density" value="${mat_density * wh_density_factor}" />
-    <xacro:property name="wh_radius"  value="${0.020 * SCALE}" />
+    <xacro:property name="wh_radius"  value="${$(arg wh_radius) * SCALE}" />
     <xacro:property name="wh_length"  value="${0.005 * SCALE}" />
     <xacro:property name="wh_mass"    value="${wh_density * PI * (wh_radius**2) * wh_length}" />
     <!-- Weg parameters -->
     <xacro:property name="wg_density_factor" value="0.5" />
-    <xacro:property name="wg_density" value="${mat_density * wg_density_factor}" />
-    <xacro:property name="wg_length"  value="${wh_radius * 0.75}" />
-    <xacro:property name="wg_width"   value="${0.001 * SCALE}" />
-    <xacro:property name="wg_height"  value="${0.002 * SCALE}" />
-    <xacro:property name="wg_mass"    value="${wg_density * wg_length * wg_width * wg_height}" />
+    <xacro:property name="wg_density"   value="${mat_density * wg_density_factor}" />
+    <xacro:property name="wg_length"    value="${wh_radius * 0.75}" />
+    <xacro:property name="wg_width"     value="${0.001 * SCALE}" />
+    <xacro:property name="wg_height"    value="${0.002 * SCALE}" />
+    <xacro:property name="wg_mass"      value="${wg_density * wg_length * wg_width * wg_height}" />
+    <xacro:property name="wg_per_wheel" value="$(arg wg_per_wheel)" />
     <!-- Weg tip parameters -->
     <xacro:property name="wt_density_factor" value="0.5" />

Commit message: Changed xacro arguments back to absolute sizes and them to the parameter server.

File: adabot_description/urdf/adabot.macros.xacro (robot description, xacro)
@@ -157,9 +157,8 @@
         <!-- Connect the weg to the wheel with a prismatic joint -->
         <joint name="${weg_name}_joint" type="prismatic">
-        <!-- <joint name="${weg_name}_joint" type="fixed"> -->
             <parent link="${parent}" />
             <child link="${weg_name}" />
             <origin xyz="0 0 0" rpy="0 ${2 * PI * (number/total)} 0" />
-            <limit upper="${wh_radius * 0.7}" lower="0" effort="100" velocity="10" />
+            <limit upper="${wg_length}" lower="0" effort="100" velocity="10" />
         </joint>
         <!--

File: adabot_description/urdf/adabot.parameters.xacro (robot description, xacro)
@@ -4,11 +4,12 @@
          Command line arguments for the adabot
     -->
-    <!-- These are factors so that they place nice with scaling -->
-    <xacro:arg name="ch_length_factor"    default="1" />
-    <xacro:arg name="ch_width_factor"     default="1" />
-    <xacro:arg name="wh_radius_factor"    default="1" />
+    <!-- Dimensions of the robot (these will be scaled) -->
+    <xacro:arg name="ch_length"    default="0.070" />
+    <xacro:arg name="ch_width"     default="0.100" />
+    <xacro:arg name="wh_radius"    default="0.020" />
+    <xacro:arg name="ax_radius"    default="0.008" />
     <!-- Number of wegs per wheel -->
     <xacro:arg name="wg_per_wheel" default="5" />
-    <!-- Global size scaling factor -->
+    <!-- Global size scaling parameter -->
     <xacro:arg name="scale"        default="4" />
     <!--
@@ -22,6 +23,6 @@
     <xacro:property name="ch_density_factor" value="0.4" />
     <xacro:property name="ch_density" value="${mat_density * ch_density_factor}" />
-    <xacro:property name="ch_length"  value="${0.100 * $(arg ch_length_factor) * SCALE}" />
-    <xacro:property name="ch_width"   value="${0.070 * $(arg ch_width_factor) * SCALE}" />
+    <xacro:property name="ch_length"  value="${$(arg ch_length) * SCALE}" />
+    <xacro:property name="ch_width"   value="${$(arg ch_width) * SCALE}" />
     <xacro:property name="ch_height"  value="${0.025 * SCALE}" />
     <xacro:property name="ch_mass"    value="${ch_density * ch_length * ch_width * ch_height}" />
@@ -29,11 +30,12 @@
     <xacro:property name="wh_density_factor" value="0.1" />
     <xacro:property name="wh_density" value="${mat_density * wh_density_factor}" />
-    <xacro:property name="wh_radius"  value="${0.020 * $(arg wh_radius_factor) * SCALE}" />
+    <xacro:property name="wh_radius"  value="${$(arg wh_radius) * SCALE}" />
     <xacro:property name="wh_length"  value="${0.005 * SCALE}" />
     <xacro:property name="wh_mass"    value="${wh_density * PI * (wh_radius**2) * wh_length}" />
     <!-- Weg parameters -->
+    <xacro:property name="ax_radius" value="${$(arg ax_radius) * SCALE}" />
     <xacro:property name="wg_density_factor" value="0.5" />
     <xacro:property name="wg_density"   value="${mat_density * wg_density_factor}" />
-    <xacro:property name="wg_length"    value="${wh_radius * 0.75}" />
+    <xacro:property name="wg_length"    value="${wh_radius - ax_radius}" />
     <xacro:property name="wg_width"     value="${0.001 * SCALE}" />
     <xacro:property name="wg_height"    value="${0.002 * SCALE}" />

Commit message: Updated visuals.

File: adabot_description/urdf/adabot.macros.xacro (robot description, xacro)
@@ -33,5 +33,13 @@
         <link name="${wheel_name}">
             <visual>
-                <xacro:insert_block name="wheel_geometry" />
+                <!-- <xacro:insert_block name="wheel_geometry" /> -->
+                <!-- <origin xyz="0 0 0" rpy="${PI/2} 0 0" />
+                <geometry>
+                    <cylinder length="${wh_length}" radius="${wh_radius}" />
+                </geometry> -->
+                <origin xyz="0 0 0" rpy="0 0 0" />
+                <geometry>
+                    <mesh filename="package://adabot_description/meshes/wheel.stl" scale="0.004 0.004 0.004" />
+                </geometry>
                 <material name="black" />
             </visual>
@@ -137,5 +145,9 @@
         <link name="${weg_name}">
             <visual>
-                <xacro:insert_block name="weg_geometry" />
+                <!-- <xacro:insert_block name="weg_geometry" /> -->
+                <origin xyz="0.024 0 0" rpy="0 ${PI/2} ${-PI/2}" />
+                <geometry>
+                    <mesh filename="package://adabot_description/meshes/weg.stl" scale="0.004 0.004 0.004" />
+                </geometry>
                 <material name="white" />
             </visual>
@@ -183,8 +195,11 @@
         <!-- Attach a sphere to the end of the weg for better physics (less jitter) -->
         <link name="${weg_name}_tip">
-            <visual>
+            <!-- <visual>
                 <xacro:insert_block name="weg_tip_geometry" />
+                <geometry>
+                    <sphere radius="${wt_radius * 0.5}" />
+                </geometry>
                 <material name="black" />
-            </visual>
+            </visual> -->
             <collision>
                 <xacro:insert_block name="weg_tip_geometry" />

File: adabot_description/urdf/adabot.main.xacro (robot description, xacro)
@@ -14,5 +14,9 @@
     <link name="chassis">
         <visual>
-            <xacro:insert_block name="chassis_geometry" />
+            <!-- <xacro:insert_block name="chassis_geometry" /> -->
+            <origin xyz="0 0 0" rpy="${PI/2} 0 ${PI/2}" />
+            <geometry>
+                <mesh filename="package://adabot_description/meshes/chassis.stl" scale="0.004 0.004 0.004" />
+            </geometry>
             <material name="white" />
         </visual>
@@ -44,10 +48,10 @@
     <!-- Add a roll cage -->
     <link name="chassis_cage">
-        <visual>
+        <!-- <visual>
             <origin xyz="0 0 0" rpy="0 0 0" />
             <geometry>
                 <sphere radius="${cg_radius}" />
             </geometry>
-        </visual>
+        </visual> -->
         <collision>
             <origin xyz="0 0 0" rpy="0 0 0" />

Commit message: Creating a visual debug mode

File: adabot_description/urdf/adabot.macros.xacro (robot description, xacro)
@@ -1,20 +1,4 @@
 <?xml version="1.0"?>
 <robot xmlns:xacro="http://www.ros.org/wiki/xacro" name="adabot">
-    <!-- Create the chassis geometry (for visuals and collisions) -->
-    <xacro:property name="chassis_geometry">
-        <origin xyz="0 0 0" rpy="0 0 0" />
-        <geometry>
-            <box size="${ch_length} ${ch_width} ${ch_height}" />
-        </geometry>
-    </xacro:property>
-    <!-- Create the wheel geometry (for visuals and collisions) -->
-    <xacro:property name="wheel_geometry">
-        <!-- Cylinders default with their height along the z axis -->
-        <origin xyz="0 0 0" rpy="${PI/2} 0 0" />
-        <geometry>
-            <!-- <cylinder length="${wh_length}" radius="${wh_radius}" /> -->
-            <sphere radius="${wh_radius}" />
-        </geometry>
-    </xacro:property>
     <!--
          Macro for creating wheels
@@ -26,4 +10,13 @@
         <!-- The name of the current wheel -->
         <xacro:property name="wheel_name" value="${suffix}_wheel" />
+        <!-- Create the wheel geometry (for visual debug and collisions) -->
+        <xacro:property name="wheel_geometry">
+            <!-- Cylinders default with their height along the z axis -->
+            <origin xyz="0 0 0" rpy="${PI/2} 0 0" />
+            <geometry>
+                <!-- <cylinder length="${wh_length}" radius="${wh_radius}" /> -->
+                <sphere radius="${wh_radius}" />
+            </geometry>
+        </xacro:property>
         <!-- Add the wheel's Gazebo material -->
         <xacro:gz_black_material name="${wheel_name}" />
@@ -33,13 +26,13 @@
         <link name="${wheel_name}">
             <visual>
-                <!-- <xacro:insert_block name="wheel_geometry" /> -->
-                <!-- <origin xyz="0 0 0" rpy="${PI/2} 0 0" />
-                <geometry>
-                    <cylinder length="${wh_length}" radius="${wh_radius}" />
-                </geometry> -->
-                <origin xyz="0 0 0" rpy="0 0 0" />
-                <geometry>
-                    <mesh filename="package://adabot_description/meshes/wheel.stl" scale="0.004 0.004 0.004" />
-                </geometry>
+                <xacro:if value="${debug_visual == 'true'}">
+                    <xacro:insert_block name="wheel_geometry" />
+                </xacro:if>
+                <xacro:if value="${debug_visual == 'false'}">
+                    <origin xyz="0 0 0" rpy="0 0 0" />
+                    <geometry>
+                        <mesh filename="package://adabot_description/meshes/wheel.stl" scale="0.004 0.004 0.004" />
+                    </geometry>
+                </xacro:if>
                 <material name="black" />
             </visual>
@@ -112,19 +105,4 @@
         </xacro:if>
     </xacro:macro>
-    <!-- Create the weg geometry (for visuals and collisions) -->
-    <xacro:property name="weg_geometry">
-        <origin xyz="${wh_radius/2} 0 0" rpy="0 0 0" />
-        <!-- <origin xyz="${wh_radius} 0 0" rpy="0 0 0" /> -->
-        <geometry>
-            <box size="${wg_length} ${wg_width} ${wg_height}" />
-        </geometry>
-    </xacro:property>
-    <!-- Create a geometry for the weg tip -->
-    <xacro:property name="weg_tip_geometry">
-        <!-- <origin xyz="${wh_radius} 0 0" rpy="0 0 0" /> -->
-        <geometry>
-            <sphere radius="${wt_radius}" />
-        </geometry>
-    </xacro:property>
     <!--
          Macro for creating wegs
@@ -137,4 +115,19 @@
         <!-- The name of the current weg (based on the parent wheel's name) -->
         <xacro:property name="weg_name" value="${wheel}_weg_${number}" />
+        <!-- Create the weg geometry (for visuals and collisions) -->
+        <xacro:property name="weg_geometry">
+            <origin xyz="${wh_radius/2} 0 0" rpy="0 0 0" />
+            <!-- <origin xyz="${wh_radius} 0 0" rpy="0 0 0" /> -->
+            <geometry>
+                <box size="${wg_length} ${wg_width} ${wg_height}" />
+            </geometry>
+        </xacro:property>
+        <!-- Create a geometry for the weg tip -->
+        <xacro:property name="weg_tip_geometry">
+            <!-- <origin xyz="${wh_radius} 0 0" rpy="0 0 0" /> -->
+            <geometry>
+                <sphere radius="${wt_radius}" />
+            </geometry>
+        </xacro:property>
         <!-- Add the weg's Gazebo material -->
         <xacro:gz_white_material name="${weg_name}" />
@@ -145,9 +138,13 @@
         <link name="${weg_name}">
             <visual>
-                <!-- <xacro:insert_block name="weg_geometry" /> -->
-                <origin xyz="0.024 0 0" rpy="0 ${PI/2} ${-PI/2}" />
-                <geometry>
-                    <mesh filename="package://adabot_description/meshes/weg.stl" scale="0.004 0.004 0.004" />
-                </geometry>
+                <xacro:if value="${debug_visual == 'true'}">
+                    <xacro:insert_block name="weg_geometry" />
+                </xacro:if>
+                <xacro:if value="${debug_visual == 'false'}">
+                    <origin xyz="0.024 0 0" rpy="0 ${PI/2} ${-PI/2}" />
+                    <geometry>
+                        <mesh filename="package://adabot_description/meshes/weg.stl" scale="0.004 0.004 0.004" />
+                    </geometry>
+                </xacro:if>
                 <material name="white" />
             </visual>
@@ -195,11 +192,10 @@
         <!-- Attach a sphere to the end of the weg for better physics (less jitter) -->
         <link name="${weg_name}_tip">
-            <!-- <visual>
-                <xacro:insert_block name="weg_tip_geometry" />
-                <geometry>
-                    <sphere radius="${wt_radius * 0.5}" />
-                </geometry>
-                <material name="black" />
-            </visual> -->
+            <xacro:if value="${debug_visual == 'true'}">
+                <visual>
+                    <xacro:insert_block name="weg_tip_geometry" />
+                    <material name="black" />
+                </visual>
+            </xacro:if>
             <collision>
                 <xacro:insert_block name="weg_tip_geometry" />

File: adabot_description/urdf/adabot.main.xacro (robot description, xacro)
@@ -9,4 +9,11 @@
     <!-- Add the Gazebo related elements -->
     <xacro:include filename="$(find adabot_description)/urdf/adabot.gazebo.xacro" />
+    <!-- Create the chassis geometry (for visual debug and collisions) -->
+    <xacro:property name="chassis_geometry">
+        <origin xyz="0 0 0" rpy="0 0 0" />
+        <geometry>
+            <box size="${ch_length} ${ch_width} ${ch_height}" />
+        </geometry>
+    </xacro:property>
     <!-- Add the base_link and the chassis. The base_link helps with positioning. -->
     <link name="base_link" />
@@ -14,9 +21,13 @@
     <link name="chassis">
         <visual>
-            <!-- <xacro:insert_block name="chassis_geometry" /> -->
-            <origin xyz="0 0 0" rpy="${PI/2} 0 ${PI/2}" />
-            <geometry>
-                <mesh filename="package://adabot_description/meshes/chassis.stl" scale="0.004 0.004 0.004" />
-            </geometry>
+            <xacro:if value="${debug_visual == 'true'}">
+                <xacro:insert_block name="chassis_geometry" />
+            </xacro:if>
+            <xacro:if value="${debug_visual == 'false'}">
+                <origin xyz="0 0 0" rpy="${PI/2} 0 ${PI/2}" />
+                <geometry>
+                    <mesh filename="package://adabot_description/meshes/chassis.stl" scale="0.004 0.004 0.004" />
+                </geometry>
+            </xacro:if>
             <material name="white" />
         </visual>
@@ -46,17 +57,20 @@
     <xacro:wheel reflect_lr="1"  reflect_fr="-1" suffix="rear_left"   />
     <xacro:wheel reflect_lr="-1" reflect_fr="-1" suffix="rear_right"  />
+    <!-- Create the roll cage (for visual debug and collisions) -->
+    <xacro:property name="roll_cage_geometry">
+        <origin xyz="0 0 0" rpy="0 0 0" />
+        <geometry>
+            <sphere radius="${cg_radius}" />
+        </geometry>
+    </xacro:property>
     <!-- Add a roll cage -->
     <link name="chassis_cage">
-        <!-- <visual>
-            <origin xyz="0 0 0" rpy="0 0 0" />
-            <geometry>
-                <sphere radius="${cg_radius}" />
-            </geometry>
-        </visual> -->
+        <xacro:if value="${debug_visual == 'true'}">
+            <visual>
+                <xacro:insert_block name="roll_cage_geometry" />
+            </visual>
+        </xacro:if>
         <collision>
-            <origin xyz="0 0 0" rpy="0 0 0" />
-            <geometry>
-                <sphere radius="${cg_radius}" />
-            </geometry>
+            <xacro:insert_block name="roll_cage_geometry" />
         </collision>
         <inertial>

File: adabot_description/urdf/adabot.parameters.xacro (robot description, xacro)
@@ -13,4 +13,6 @@
     <!-- Global size scaling parameter -->
     <xacro:arg name="scale"        default="4" />
+    <!-- Visual debug mode -->
+    <xacro:arg name="debug_visual" default="false" />
     <!--
          Properties for the robot bodies
@@ -53,3 +55,5 @@
     <!-- Vertical offset so that the robot starts above ground -->
     <xacro:property name="z_offset" value="${wh_radius * 2}" />
+    <!-- Visual debug mode -->
+    <xacro:property name="debug_visual" value="$(arg debug_visual)" />
 </robot>
