Commit message: Added scale to mesh calls. Removed debug_visual from server storage. Removed commented code.

File: adabot_description/urdf/adabot.macros.xacro (robot description, xacro)
@@ -12,8 +12,6 @@
         <!-- Create the wheel geometry (for visual debug and collisions) -->
         <xacro:property name="wheel_geometry">
-            <!-- Cylinders default with their height along the z axis -->
             <origin xyz="0 0 0" rpy="${PI/2} 0 0" />
             <geometry>
-                <!-- <cylinder length="${wh_length}" radius="${wh_radius}" /> -->
                 <sphere radius="${wh_radius}" />
             </geometry>
@@ -32,5 +30,6 @@
                     <origin xyz="0 0 0" rpy="0 0 0" />
                     <geometry>
-                        <mesh filename="package://adabot_description/meshes/wheel.stl" scale="0.004 0.004 0.004" />
+                        <mesh filename="package://adabot_description/meshes/wheel.stl"
+                                scale="${0.001 * SCALE} ${0.001 * SCALE} ${0.001 * SCALE}" />
                     </geometry>
                 </xacro:if>
@@ -118,5 +117,4 @@
         <xacro:property name="weg_geometry">
             <origin xyz="${wh_radius/2} 0 0" rpy="0 0 0" />
-            <!-- <origin xyz="${wh_radius} 0 0" rpy="0 0 0" /> -->
             <geometry>
                 <box size="${wg_length} ${wg_width} ${wg_height}" />
@@ -125,5 +123,4 @@
         <!-- Create a geometry for the weg tip -->
         <xacro:property name="weg_tip_geometry">
-            <!-- <origin xyz="${wh_radius} 0 0" rpy="0 0 0" /> -->
             <geometry>
                 <sphere radius="${wt_radius}" />
@@ -144,5 +141,6 @@
                     <origin xyz="0.024 0 0" rpy="0 ${PI/2} ${-PI/2}" />
                     <geometry>
-                        <mesh filename="package://adabot_description/meshes/weg.stl" scale="0.004 0.004 0.004" />
+                        <mesh filename="package://adabot_description/meshes/weg.stl"
+                                scale="${0.001 * SCALE} ${0.001 * SCALE} ${0.001 * SCALE}" />
                     </geometry>
                 </xacro:if>

File: adabot_description/urdf/adabot.main.xacro (robot description, xacro)
@@ -27,5 +27,6 @@
                 <origin xyz="0 0 0" rpy="${PI/2} 0 ${PI/2}" />
                 <geometry>
-                    <mesh filename="package://adabot_description/meshes/chassis.stl" scale="0.004 0.004 0.004" />
+                    <mesh filename="package://adabot_description/meshes/chassis.stl"
+                          scale="${0.001 * SCALE} ${0.001 * SCALE} ${0.001 * SCALE}" />
                 </geometry>
             </xacro:if>

Commit message: Changed `debug_visual` to `debug_visuals`

File: adabot_description/urdf/adabot.macros.xacro (robot description, xacro)
@@ -24,8 +24,8 @@
         <link name="${wheel_name}">
             <visual>
-                <xacro:if value="${debug_visual == 'true'}">
+                <xacro:if value="${debug_visuals == 'true'}">
                     <xacro:insert_block name="wheel_geometry" />
                 </xacro:if>
-                <xacro:if value="${debug_visual == 'false'}">
+                <xacro:if value="${debug_visuals == 'false'}">
                     <origin xyz="0 0 0" rpy="0 0 0" />
                     <geometry>
@@ -135,8 +135,8 @@
         <link name="${weg_name}">
             <visual>
-                <xacro:if value="${debug_visual == 'true'}">
+                <xacro:if value="${debug_visuals == 'true'}">
                     <xacro:insert_block name="weg_geometry" />
                 </xacro:if>
-                <xacro:if value="${debug_visual == 'false'}">
+                <xacro:if value="${debug_visuals == 'false'}">
                     <origin xyz="0.024 0 0" rpy="0 ${PI/2} ${-PI/2}" />
                     <geometry>
@@ -190,5 +190,5 @@
         <!-- Attach a sphere to the end of the weg for better physics (less jitter) -->
         <link name="${weg_name}_tip">
-            <xacro:if value="${debug_visual == 'true'}">
+            <xacro:if value="${debug_visuals == 'true'}">
                 <visual>
                     <xacro:insert_block name="weg_tip_geometry" />

File: adabot_description/urdf/adabot.main.xacro (robot description, xacro)
@@ -21,8 +21,8 @@
     <link name="chassis">
         <visual>
-            <xacro:if value="${debug_visual == 'true'}">
+            <xacro:if value="${debug_visuals == 'true'}">
                 <xacro:insert_block name="chassis_geometry" />
             </xacro:if>
-            <xacro:if value="${debug_visual == 'false'}">
+            <xacro:if value="${debug_visuals == 'false'}">
                 <origin xyz="0 0 0" rpy="${PI/2} 0 ${PI/2}" />
                 <geometry>
@@ -67,5 +67,5 @@
     <!-- Add a roll cage -->
     <link name="chassis_cage">
-        <xacro:if value="${debug_visual == 'true'}">
+        <xacro:if value="${debug_visuals == 'true'}">
             <visual>
                 <xacro:insert_block name="roll_cage_geometry" />

File: adabot_description/urdf/adabot.parameters.xacro (robot description, xacro)
@@ -5,14 +5,14 @@
     -->
     <!-- Dimensions of the robot (these will be scaled) -->
-    <xacro:arg name="ch_length"    default="0.070" />
-    <xacro:arg name="ch_width"     default="0.100" />
-    <xacro:arg name="wh_radius"    default="0.020" />
-    <xacro:arg name="ax_radius"    default="0.008" />
+    <xacro:arg name="ch_length"     default="0.070" />
+    <xacro:arg name="ch_width"      default="0.100" />
+    <xacro:arg name="wh_radius"     default="0.020" />
+    <xacro:arg name="ax_radius"     default="0.008" />
     <!-- Number of wegs per wheel -->
-    <xacro:arg name="wg_per_wheel" default="5" />
+    <xacro:arg name="wg_per_wheel"  default="5" />
     <!-- Global size scaling parameter -->
-    <xacro:arg name="scale"        default="4" />
+    <xacro:arg name="scale"         default="4" />
     <!-- Visual debug mode -->
-    <xacro:arg name="debug_visual" default="false" />
+    <xacro:arg name="debug_visuals" default="false" />
     <!--
          Properties for the robot bodies
@@ -56,4 +56,4 @@
     <xacro:property name="z_offset" value="${wh_radius * 2}" />
     <!-- Visual debug mode -->
-    <xacro:property name="debug_visual" value="$(arg debug_visual)" />
+    <xacro:property name="debug_visuals" value="$(arg debug_visuals)" />
 </robot>
