Commit message: Added instructions to the gazebo XACRO file.

File: adabot_description/urdf/adabot.gazebo.xacro (robot description, xacro)
@@ -1,3 +1,44 @@
 <?xml version="1.0"?>
 <robot xmlns:xacro="http://www.ros.org/wiki/xacro" name="adabot">
+    <!--
+        Gazebo requires the following:
+            An <inertia> element within each <link> (handled in adabot.main.xacro).
+        It also useful to specify the following:
+            A <gazebo> element for every <link>
+                - Gazebo colors
+                - DAE files for textures
+                - sensor plugins
+            A <gazebo> element for every <joint>
+                - damping dynamics
+                - actuator plugins
+            A <link name="world" /> if the robot is rigidyly attached to the world
+        By conventions, units should be specified in meters and kilograms.
+    -->
+    <gazebo reference="${chassisname}">
+        <material>Gazebo/White</material>
+    </gazebo>
+    <!-- Add colors for other links -->
+    <!-- Add simulated IMU:
+            gazeborosimu
+            gazeborosimusensor <-- probably this one
+    -->
+    <!-- Add simulated wheel encoders -->
+    <!-- Add wheel motors and control -->
+    <!-- Add linear servo motors and control -->
+<!--     <gazebo>
+        <plugin name="skid_steer_drive_controller" filename="libgazebo_ros_skid_steer_drive.so">
+            <updateRate>100.0</updateRate>
+            <robotNamespace>/</robotNamespace>
+            <leftFrontJoint>front_left_wheel_joint</leftFrontJoint>
+            <rightFrontJoint>front_right_wheel_joint</rightFrontJoint>
+            <leftRearJoint>back_left_wheel_joint</leftRearJoint>
+            <rightRearJoint>back_right_wheel_joint</rightRearJoint>
+            <wheelSeparation>0.4</wheelSeparation>
+            <wheelDiameter>0.215</wheelDiameter>
+            <robotBaseFrame>base_link</robotBaseFrame>
+            <torque>20</torque>
+            <topicName>cmd_vel</topicName>
+            <broadcastTF>false</broadcastTF>
+        </plugin>
+    </gazebo> -->
 </robot>

Commit message: Added the adabot_control package. Currently working on getting the velocity controller working (position control works).

File: adabot_description/urdf/adabot.gazebo.xacro (robot description, xacro)
@@ -18,8 +18,18 @@
         <material>Gazebo/White</material>
     </gazebo>
+    <xacro:macro name="gz_wheel_material" params="name">
+        <gazebo reference="${name}">
+            <material>Gazebo/Black</material>
+        </gazebo>
+    </xacro:macro>
+    <gazebo>
+        <plugin name="gazebo_ros_control" filename="libgazebo_ros_control.so">
+            <robotNamespace>/adabot</robotNamespace>
+        </plugin>
+    </gazebo>
     <!-- Add colors for other links -->
     <!-- Add simulated IMU:
             gazeborosimu
-            gazeborosimusensor <-- probably this one
+            gazeborosimusensor  *probably this one*
     -->
     <!-- Add simulated wheel encoders -->

File: adabot_description/urdf/adabot.main.xacro (robot description, xacro)
@@ -4,25 +4,26 @@
          Properties for the robot bodies
     -->
-    <xacro:property name="PI" value="3.1415926535897931"/>
+    <xacro:property name="PI" value="3.1415926535897931 "/>
+    <xacro:property name="SCALE" value="2" />
     <!-- Typical density of plastics -->
     <xacro:property name="mat_density" value="1000.0" />
     <!-- Wheel parameters -->
-    <xacro:property name="wh_radius" value="0.02" />
-    <xacro:property name="wh_length" value="0.005" />
-    <xacro:property name="wh_mass" value="${mat_density*PI*(wh_radius**2)*wh_length}" />
+    <xacro:property name="wh_radius" value="${0.020 * SCALE}" />
+    <xacro:property name="wh_length" value="${0.005 * SCALE}" />
+    <xacro:property name="wh_mass"   value="${mat_density*PI*(wh_radius**2)*wh_length}" />
     <!-- Axle parameters -->
     <xacro:property name="ax_axis" value="0 1 0" />
     <!-- Chassis parameters -->
-    <xacro:property name="ch_length" value="0.1" />
-    <xacro:property name="ch_width" value="0.07" />
-    <xacro:property name="ch_height" value="0.035" />
-    <xacro:property name="ch_mass" value="${mat_density*ch_length*ch_width*ch_height}" />
+    <xacro:property name="ch_length" value="${0.100 * SCALE}" />
+    <xacro:property name="ch_width"  value="${0.070 * SCALE}" />
+    <xacro:property name="ch_height" value="${0.035 * SCALE}" />
+    <xacro:property name="ch_mass"   value="${mat_density*ch_length*ch_width*ch_height}" />
     <!-- Weg parameters -->
     <xacro:property name="wg_length" value="${wh_radius*2}" />
-    <xacro:property name="wg_width" value="0.001" />
-    <xacro:property name="wg_height" value="0.002" />
-    <xacro:property name="wg_mass" value="${mat_density*wg_length*wg_width*wg_height}" />
+    <xacro:property name="wg_width"  value="${0.001 * SCALE}" />
+    <xacro:property name="wg_height" value="${0.002 * SCALE}" />
+    <xacro:property name="wg_mass"   value="${mat_density*wg_length*wg_width*wg_height}" />
     <!-- Vertical offset so that the robot starts above ground -->
-    <xacro:property name="zoffset" value="${wh_radius*1.1/2}" />
+    <xacro:property name="zoffset" value="${wh_radius*1.1/2 * 10}" />
     <!--
          Properties for names, colors, and Gazebo
@@ -51,5 +52,5 @@
     -->
     <xacro:macro name="weg" params="wheel number parent total">
-        <xacro:property name="wg_name" value="wg-${wheel}-${number}" />
+        <xacro:property name="wg_name" value="wg_${wheel}_${number}" />
         <link name="${wg_name}">
             <visual>
@@ -72,5 +73,5 @@
             </inertial>
         </link>
-        <joint name="${wg_name}-joint" type="prismatic">
+        <joint name="${wg_name}_joint" type="prismatic">
             <parent link="${parent}" />
             <child link="${wg_name}" />
@@ -97,5 +98,6 @@
     -->
     <xacro:macro name="wheel" params="reflect_lr reflect_fb suffix parent">
-        <xacro:property name="wh_name" value="wh-${suffix}" />
+        <xacro:property name="wh_name" value="wh_${suffix}" />
+        <xacro:gz_wheel_material name="${wh_name}" />
         <link name="${wh_name}">
             <visual>
@@ -108,4 +110,5 @@
             <inertial>
                 <mass value="${wh_mass}" />
+                <origin rpy="1.57075 0 0" xyz="0 0 0" />
                 <inertia
                     ixx="${(1/12)*wh_mass*(3*wh_radius**2 + wh_length**2)}"
@@ -118,5 +121,5 @@
             </inertial>
         </link>
-        <joint name="ax-${suffix}" type="continuous">
+        <joint name="ax_${suffix}" type="continuous">
             <parent link="${parent}" />
             <child link="${wh_name}" />
@@ -159,4 +162,5 @@
         <inertial>
             <mass value="${ch_mass}" />
+            <origin xyz="0 0 ${zoffset}" rpy="0 0 0"/>
             <inertia
                 ixx="${(1/12)*ch_mass*(ch_width**2 + ch_height**2)}"
@@ -172,7 +176,23 @@
          Macro calls for creating wheels
     -->
-    <xacro:wheel reflect_lr="-1" reflect_fb="1" suffix="front-left" parent="${chassisname}" />
-    <xacro:wheel reflect_lr="1" reflect_fb="1" suffix="front-right" parent="${chassisname}" />
-    <xacro:wheel reflect_lr="-1" reflect_fb="-1" suffix="back-left" parent="${chassisname}" />
-    <xacro:wheel reflect_lr="1" reflect_fb="-1" suffix="back-right" parent="${chassisname}" />
+    <xacro:wheel reflect_lr="-1" reflect_fb="1" suffix="front_left" parent="${chassisname}" />
+    <xacro:wheel reflect_lr="1" reflect_fb="1" suffix="front_right" parent="${chassisname}" />
+    <xacro:wheel reflect_lr="-1" reflect_fb="-1" suffix="back_left" parent="${chassisname}" />
+    <xacro:wheel reflect_lr="1" reflect_fb="-1" suffix="back_right" parent="${chassisname}" />
+    <!--
+         Add a transmission for ros_control so that it can control the wheel motors
+    -->
+    <transmission name="tran1">
+        <type>transmission_interface/SimpleTransmission</type>
+        <joint name="ax_front_left">
+            <hardwareInterface>hardware_interface/EffortJointInterface</hardwareInterface>
+        </joint>
+        <actuator name="motor1">
+            <hardwareInterface>hardware_interface/EffortJointInterface</hardwareInterface>
+            <mechanicalReduction>1</mechanicalReduction>
+        </actuator>
+    </transmission>
+    <!--
+         Add a Gazebo world element as a reference
+    -->
 </robot>

Commit message: Updating the xacro files to reposition the link frame of the chassis (it will end up at the COM).

File: adabot_description/urdf/adabot.gazebo.xacro (robot description, xacro)
@@ -15,5 +15,5 @@
         By conventions, units should be specified in meters and kilograms.
     -->
-    <gazebo reference="${chassisname}">
+    <gazebo reference="chassis">
         <material>Gazebo/White</material>
     </gazebo>
@@ -26,4 +26,5 @@
         <plugin name="gazebo_ros_control" filename="libgazebo_ros_control.so">
             <robotNamespace>/adabot</robotNamespace>
+            <robotSimType>gazebo_ros_control/DefaultRobotHWSim</robotSimType>
         </plugin>
     </gazebo>

File: adabot_description/urdf/adabot.main.xacro (robot description, xacro)
@@ -8,20 +8,24 @@
     <!-- Typical density of plastics -->
     <xacro:property name="mat_density" value="1000.0" />
+    <!-- Chassis parameters -->
+    <xacro:property name="ch_density_factor" value="0.4" />
+    <xacro:property name="ch_density" value="${mat_density * ch_density_factor}" />
+    <xacro:property name="ch_length"  value="${0.100 * SCALE}" />
+    <xacro:property name="ch_width"   value="${0.070 * SCALE}" />
+    <xacro:property name="ch_height"  value="${0.035 * SCALE}" />
+    <xacro:property name="ch_mass"    value="${ch_density * ch_length * ch_width * ch_height}" />
     <!-- Wheel parameters -->
-    <xacro:property name="wh_radius" value="${0.020 * SCALE}" />
-    <xacro:property name="wh_length" value="${0.005 * SCALE}" />
-    <xacro:property name="wh_mass"   value="${mat_density*PI*(wh_radius**2)*wh_length}" />
-    <!-- Axle parameters -->
-    <xacro:property name="ax_axis" value="0 1 0" />
-    <!-- Chassis parameters -->
-    <xacro:property name="ch_length" value="${0.100 * SCALE}" />
-    <xacro:property name="ch_width"  value="${0.070 * SCALE}" />
-    <xacro:property name="ch_height" value="${0.035 * SCALE}" />
-    <xacro:property name="ch_mass"   value="${mat_density*ch_length*ch_width*ch_height}" />
+    <xacro:property name="wh_density_factor" value="0.4" />
+    <xacro:property name="wh_density" value="${mat_density * wh_density_factor}" />
+    <xacro:property name="wh_radius"  value="${0.020 * SCALE}" />
+    <xacro:property name="wh_length"  value="${0.005 * SCALE}" />
+    <xacro:property name="wh_mass"    value="${wh_density * PI * (wh_radius**2) * wh_length}" />
     <!-- Weg parameters -->
     <xacro:property name="wg_length" value="${wh_radius*2}" />
     <xacro:property name="wg_width"  value="${0.001 * SCALE}" />
     <xacro:property name="wg_height" value="${0.002 * SCALE}" />
-    <xacro:property name="wg_mass"   value="${mat_density*wg_length*wg_width*wg_height}" />
+    <xacro:property name="wg_mass"   value="${mat_density * wg_length * wg_width * wg_height}" />
+    <!-- Axle parameters -->
+    <xacro:property name="ax_axis" value="0 1 0" />
     <!-- Vertical offset so that the robot starts above ground -->
     <xacro:property name="zoffset" value="${wh_radius*1.1/2 * 10}" />
@@ -29,6 +33,4 @@
          Properties for names, colors, and Gazebo
     -->
-    <!-- The chassis is the parent of several other links, so we need it's name -->
-    <xacro:property name="chassisname" value="base_link" />
     <!-- Import colors defined for Rviz -->
     <xacro:include filename="$(find adabot_description)/urdf/adabot.materials.xacro" />
@@ -124,5 +126,6 @@
             <parent link="${parent}" />
             <child link="${wh_name}" />
-            <origin rpy="0 0 0" xyz="${ch_length/2*reflect_fb} ${(wh_length+ch_width)/2*reflect_lr} ${zoffset}" />
+            <!-- <origin rpy="0 0 0" xyz="${ch_length/2*reflect_fb} ${(wh_length+ch_width)/2*reflect_lr} ${zoffset}" /> -->
+            <origin rpy="0 0 0" xyz="${ch_length/2*reflect_fb} ${(wh_length+ch_width)/2*reflect_lr} 0" />
             <axis xyz="${ax_axis}" />
         </joint>
@@ -144,5 +147,6 @@
     -->
     <xacro:property name="ch_orig_geom">
-        <origin rpy="0 0 0" xyz="0 0 ${zoffset}" />
+        <!-- <origin rpy="0 0 0" xyz="0 0 ${zoffset}" /> -->
+        <origin rpy="0 0 0" xyz="0 0 0" />
         <geometry>
             <box size="${ch_length} ${ch_width} ${ch_height}" />
@@ -151,6 +155,10 @@
     <!--
          The main chassis/body
-    -->
-    <link name="${chassisname}">
+            Note: the chassis is connect to the world link so that it's link frame is
+            easier to visualize. This will also help when we start to include multiple
+            robots.
+    -->
+    <link name="world" />
+    <link name="chassis">
         <visual>
             <xacro:insert_block name="ch_orig_geom" />
@@ -162,5 +170,5 @@
         <inertial>
             <mass value="${ch_mass}" />
-            <origin xyz="0 0 ${zoffset}" rpy="0 0 0"/>
+            <!-- <origin xyz="0 0 ${zoffset}" rpy="0 0 0"/> -->
             <inertia
                 ixx="${(1/12)*ch_mass*(ch_width**2 + ch_height**2)}"
@@ -173,20 +181,25 @@
         </inertial>
     </link>
+    <joint name="world_joint" type="fixed">
+        <origin xyz="0 0 0" rpy="0 0 0" />
+        <parent link="world" />
+        <child link="chassis" />
+    </joint>
     <!--
          Macro calls for creating wheels
     -->
-    <xacro:wheel reflect_lr="-1" reflect_fb="1" suffix="front_left" parent="${chassisname}" />
-    <xacro:wheel reflect_lr="1" reflect_fb="1" suffix="front_right" parent="${chassisname}" />
-    <xacro:wheel reflect_lr="-1" reflect_fb="-1" suffix="back_left" parent="${chassisname}" />
-    <xacro:wheel reflect_lr="1" reflect_fb="-1" suffix="back_right" parent="${chassisname}" />
+    <xacro:wheel reflect_lr="-1" reflect_fb="1"  suffix="front_left"  parent="chassis" />
+    <xacro:wheel reflect_lr="1"  reflect_fb="1"  suffix="front_right" parent="chassis" />
+    <xacro:wheel reflect_lr="-1" reflect_fb="-1" suffix="back_left"   parent="chassis" />
+    <xacro:wheel reflect_lr="1"  reflect_fb="-1" suffix="back_right"  parent="chassis" />
     <!--
          Add a transmission for ros_control so that it can control the wheel motors
     -->
-    <transmission name="tran1">
+    <transmission name="tran_front_left" type="SimpleTransmission">
         <type>transmission_interface/SimpleTransmission</type>
         <joint name="ax_front_left">
             <hardwareInterface>hardware_interface/EffortJointInterface</hardwareInterface>
         </joint>
-        <actuator name="motor1">
+        <actuator name="motor_front_left">
             <hardwareInterface>hardware_interface/EffortJointInterface</hardwareInterface>
             <mechanicalReduction>1</mechanicalReduction>

Commit message: Mostly functional, but it has some troubles at low speeds (wheels slide instead of spin).

File: adabot_description/urdf/adabot.gazebo.xacro (robot description, xacro)
@@ -15,12 +15,4 @@
         By conventions, units should be specified in meters and kilograms.
     -->
-    <gazebo reference="chassis">
-        <material>Gazebo/White</material>
-    </gazebo>
-    <xacro:macro name="gz_wheel_material" params="name">
-        <gazebo reference="${name}">
-            <material>Gazebo/Black</material>
-        </gazebo>
-    </xacro:macro>
     <gazebo>
         <plugin name="gazebo_ros_control" filename="libgazebo_ros_control.so">
@@ -29,43 +21,31 @@
         </plugin>
     </gazebo>
-<!-- <gazebo reference="chassis">
-  <mu1 value="0.0"/>
-  <mu2 value="0.0"/>
-  <kp  value="10000000.0" />
-  <kd  value="1.0" />
-  <material>Gazebo/Blue</material>
-</gazebo>
-<gazebo reference="left_rear_wheel">
-  <mu1 value="1.0"/>
-  <mu2 value="1.0"/>
-  <kp  value="10000000.0" />
-  <kd  value="1.0" />
-  <fdir1 value="1 0 0"/>
-  <material>Gazebo/Black</material>
-</gazebo>
-<gazebo reference="right_rear_wheel">
-  <mu1 value="1.0"/>
-  <mu2 value="1.0"/>
-  <kp  value="10000000.0" />
-  <kd  value="1.0" />
-  <fdir1 value="1 0 0"/>
-  <material>Gazebo/Black</material>
-</gazebo>
-<gazebo reference="left_front_wheel">
-  <mu1 value="1.0"/>
-  <mu2 value="1.0"/>
-  <kp  value="10000000.0" />
-  <kd  value="1.0" />
-  <fdir1 value="0 0 1"/>
-  <material>Gazebo/Black</material>
-</gazebo>
-<gazebo reference="right_front_wheel">
-  <mu1 value="1.0"/>
-  <mu2 value="1.0"/>
-  <kp  value="10000000.0" />
-  <kd  value="1.0" />
-  <fdir1 value="0 0 1"/>
-  <material>Gazebo/Black</material>
-</gazebo> -->
+    <!-- http://wiki.ros.org/simulator_gazebo/Tutorials/ListOfMaterials -->
+    <xacro:macro name="gz_black_material" params="name">
+        <gazebo reference="${name}">
+            <material>Gazebo/FlatBlack</material>
+        </gazebo>
+    </xacro:macro>
+    <xacro:macro name="gz_white_material" params="name">
+        <gazebo reference="${name}">
+            <!-- <material>Gazebo/White</material> -->
+            <material>Gazebo/GreenEmissive</material>
+        </gazebo>
+    </xacro:macro>
+    <xacro:macro name="gz_blue_material" params="name">
+        <gazebo reference="${name}">
+            <material>Gazebo/Blue</material>
+        </gazebo>
+    </xacro:macro>
+    <!-- Material frictions -->
+    <xacro:macro name="gz_high_friction" params="name">
+        <gazebo reference="${name}">
+            <mu1 value="100.0"/>
+            <mu2 value="100.0"/>
+            <!-- <kp  value="10000000.0" /> -->
+            <!-- <kd  value="1.0" /> -->
+            <!-- <fdir1 value="1 0 0"/> -->
+        </gazebo>
+    </xacro:macro>
     <!-- Add colors for other links -->
     <!-- Add simulated IMU:

File: adabot_description/urdf/adabot.macros.xacro (robot description, xacro)
@@ -27,5 +27,5 @@
         <xacro:property name="wheel_name" value="${suffix}_wheel" />
         <!-- Add the wheel's Gazebo material -->
-        <xacro:gz_wheel_material name="${wheel_name}" />
+        <xacro:gz_black_material name="${wheel_name}" />
         <!-- The wheel's rigid body -->
         <link name="${wheel_name}">
@@ -105,4 +105,7 @@
         <!-- The name of the current weg (based on the parent wheel's name) -->
         <xacro:property name="weg_name" value="${wheel}_weg_${number}" />
+        <!-- Add the weg's Gazebo material -->
+        <xacro:gz_white_material name="${weg_name}" />
+        <xacro:gz_black_material name="${weg_name}_tip" />
         <!-- The weg's rigid body -->
         <link name="${weg_name}">
@@ -132,5 +135,5 @@
             <child link="${weg_name}" />
             <origin xyz="0 0 0" rpy="0 ${2 * PI * (number/total)} 0" />
-            <limit upper="${wh_radius * 0.7}" lower="0" effort="10" velocity="10" />
+            <limit upper="${wh_radius * 0.7}" lower="0" effort="100" velocity="10" />
         </joint>
         <!--
@@ -174,4 +177,6 @@
             </inertial>
         </link>
+        <!-- Make the weg tip high friction -->
+        <xacro:gz_high_friction name="${weg_name}_tip" />
         <!-- Connect the weg tip to the weg -->
         <joint name="${weg_name}_tip_joint" type="fixed">

File: adabot_description/urdf/adabot.main.xacro (robot description, xacro)
@@ -9,7 +9,8 @@
     <!-- Add the Gazebo related elements -->
     <xacro:include filename="$(find adabot_description)/urdf/adabot.gazebo.xacro" />
-    <!-- Add the base_link (needed by Gazebo) and the chassis -->
+    <!-- Add the base_link and the chassis. The base_link helps with positioning. -->
     <link name="base_link" />
     <link name="chassis">
+        <xacro:gz_white_material name="chassis" />
         <visual>
             <xacro:insert_block name="chassis_geometry" />
