Commit message: Added a simple setup for capturing video.

File: adabot_description/urdf/adabot.gazebo.xacro (robot description, xacro)
@@ -30,5 +30,5 @@
         <gazebo reference="${name}">
             <!-- <material>Gazebo/White</material> -->
-            <material>Gazebo/GreenEmissive</material>
+            <material>Gazebo/White</material>
         </gazebo>
     </xacro:macro>
@@ -41,9 +41,18 @@
     <xacro:macro name="gz_high_friction" params="name">
         <gazebo reference="${name}">
-            <mu1 value="100.0"/>
-            <mu2 value="100.0"/>
+            <mu1 value="100.0" />
+            <mu2 value="100.0" />
             <!-- <kp  value="10000000.0" /> -->
             <!-- <kd  value="1.0" /> -->
-            <!-- <fdir1 value="1 0 0"/> -->
+            <!-- <fdir1 value="1 0 0" /> -->
+        </gazebo>
+    </xacro:macro>
+    <xacro:macro name="gz_low_friction" params="name">
+        <gazebo reference="${name}">
+            <mu1 value="0.5" />
+            <mu2 value="0.5" />
+            <!-- <kp  value="10000000.0" /> -->
+            <!-- <kd  value="1.0" /> -->
+            <!-- <fdir1 value="1 0 0" /> -->
         </gazebo>
     </xacro:macro>

File: adabot_description/urdf/adabot.macros.xacro (robot description, xacro)
@@ -28,4 +28,6 @@
         <!-- Add the wheel's Gazebo material -->
         <xacro:gz_black_material name="${wheel_name}" />
+        <!-- Make the wheel have lower friction -->
+        <xacro:gz_low_friction name="${wheel_name}" />
         <!-- The wheel's rigid body -->
         <link name="${wheel_name}">
@@ -108,4 +110,6 @@
         <xacro:gz_white_material name="${weg_name}" />
         <xacro:gz_black_material name="${weg_name}_tip" />
+        <!-- Make the weg tip high friction -->
+        <xacro:gz_high_friction name="${weg_name}_tip" />
         <!-- The weg's rigid body -->
         <link name="${weg_name}">
@@ -177,6 +181,4 @@
             </inertial>
         </link>
-        <!-- Make the weg tip high friction -->
-        <xacro:gz_high_friction name="${weg_name}_tip" />
         <!-- Connect the weg tip to the weg -->
         <joint name="${weg_name}_tip_joint" type="fixed">

File: adabot_description/urdf/adabot.main.xacro (robot description, xacro)
@@ -11,6 +11,6 @@
     <!-- Add the base_link and the chassis. The base_link helps with positioning. -->
     <link name="base_link" />
+    <xacro:gz_white_material name="chassis" />
     <link name="chassis">
-        <xacro:gz_white_material name="chassis" />
         <visual>
             <xacro:insert_block name="chassis_geometry" />

File: adabot_description/urdf/adabot.materials.xacro (robot description, xacro)
@@ -2,26 +2,26 @@
 <robot xmlns:xacro="http://www.ros.org/wiki/xacro" name="adabot">
     <material name="black">
-        <color rgba="0.0 0.0 0.0 1.0"/>
+        <color rgba="0.0 0.0 0.0 1.0" />
     </material>
     <material name="blue">
-        <color rgba="0.0 0.0 0.8 1.0"/>
+        <color rgba="0.0 0.0 0.8 1.0" />
     </material>
     <material name="green">
-        <color rgba="0.0 0.8 0.0 1.0"/>
+        <color rgba="0.0 0.8 0.0 1.0" />
     </material>
     <material name="grey">
-        <color rgba="0.2 0.2 0.2 1.0"/>
+        <color rgba="0.2 0.2 0.2 1.0" />
     </material>
     <material name="orange">
-        <color rgba="${255/255} ${108/255} ${10/255} 1.0"/>
+        <color rgba="${255/255} ${108/255} ${10/255} 1.0" />
     </material>
     <material name="brown">
-        <color rgba="${222/255} ${207/255} ${195/255} 1.0"/>
+        <color rgba="${222/255} ${207/255} ${195/255} 1.0" />
     </material>
     <material name="red">
-        <color rgba="0.8 0.0 0.0 1.0"/>
+        <color rgba="0.8 0.0 0.0 1.0" />
     </material>
     <material name="white">
-        <color rgba="1.0 1.0 1.0 1.0"/>
+        <color rgba="1.0 1.0 1.0 1.0" />
     </material>
 </robot>

File: adabot_description/urdf/adabot.parameters.xacro (robot description, xacro)
@@ -4,5 +4,5 @@
          Properties for the robot bodies
     -->
-    <xacro:property name="PI" value="3.1415926535897931 "/>
+    <xacro:property name="PI" value="3.1415926535897931 " />
     <xacro:property name="SCALE" value="4" />
     <!-- Typical density of plastics -->
@@ -11,5 +11,5 @@
     <xacro:property name="ch_density_factor" value="0.4" />
     <xacro:property name="ch_density" value="${mat_density * ch_density_factor}" />
-    <xacro:property name="ch_length"  value="${0.100 * SCALE}" />
+    <xacro:property name="ch_length"  value="${0.100 * SCALE * 0.65}" />
     <xacro:property name="ch_width"   value="${0.070 * SCALE}" />
     <xacro:property name="ch_height"  value="${0.025 * SCALE}" />

Commit message: The IMU sensor has been added.

File: adabot_description/urdf/adabot.gazebo.xacro (robot description, xacro)
@@ -29,5 +29,4 @@
     <xacro:macro name="gz_white_material" params="name">
         <gazebo reference="${name}">
-            <!-- <material>Gazebo/White</material> -->
             <material>Gazebo/White</material>
         </gazebo>
@@ -57,11 +56,49 @@
         </gazebo>
     </xacro:macro>
-    <!-- Add colors for other links -->
-    <!-- Add simulated IMU:
-            gazeborosimu
-            gazeborosimusensor  *probably this one*
-    -->
-    <!-- Add simulated wheel encoders -->
-    <!-- Add wheel motors and control -->
-    <!-- Add linear servo motors and control -->
+<link name="imu_sensor_link">
+    <collision>
+        <origin xyz="0 0 0" rpy="0 0 0" />
+        <geometry>
+            <box size="0.02 0.02 0.02" />
+        </geometry>
+    </collision>
+    <visual>
+        <origin xyz="0 0 0" rpy="0 0 0" />
+        <geometry>
+            <box size="0.02 0.02 0.02" />
+        </geometry>
+        <material name="red" />
+    </visual>
+    <inertial>
+        <mass value="0.001" />
+        <origin xyz="0 0 0" rpy="0 0 0" />
+        <inertia ixx="0.00000015" ixy="0" ixz="0" iyy="0.00000015" iyz="0" izz="0.00000015" />
+    </inertial>
+</link>
+<joint name="imu_sensor_joint" type="fixed">
+    <axis xyz="0 0 1" />
+    <origin xyz="0 0 0" rpy="0 0 0" />
+    <parent link="chassis" />
+    <child link="imu_sensor_link" />
+</joint>
+<gazebo reference="imu_sensor_link">
+    <gravity>true</gravity>
+    <sensor name='imu_sensor' type='imu'>
+        <always_on>1</always_on>
+        <update_rate>100</update_rate>
+        <visualize>1</visualize>
+        <topic>__default_topic__</topic>
+        <plugin name='imu_plugin' filename='libgazebo_ros_imu_sensor.so'>
+    <frameName>imu_sensor_link</frameName>
+    <robotNamespace>/adabot</robotNamespace>
+            <topicName>imu_data</topicName>
+            <!-- <bodyName>imu_sensor_link</bodyName> -->
+            <updateRateHZ>10.0</updateRateHZ>
+            <gaussianNoise>0.0</gaussianNoise>
+            <xyzOffset>0 0 0</xyzOffset>
+            <rpyOffset>0 0 0</rpyOffset>
+        </plugin>
+        <pose>0 0 0 0 0 0</pose>
+    </sensor>
+</gazebo>
 </robot>
