Commit message: Prepend 'bot_name' to all links and joints to allow the creation of multiple adabots

File: adabot_description/urdf/adabot.gazebo.xacro (robot description, xacro)
@@ -56,49 +56,3 @@
         </gazebo>
     </xacro:macro>
-<link name="imu_sensor_link">
-    <collision>
-        <origin xyz="0 0 0" rpy="0 0 0" />
-        <geometry>
-            <box size="0.02 0.02 0.02" />
-        </geometry>
-    </collision>
-    <visual>
-        <origin xyz="0 0 0" rpy="0 0 0" />
-        <geometry>
-            <box size="0.02 0.02 0.02" />
-        </geometry>
-        <material name="red" />
-    </visual>
-    <inertial>
-        <mass value="0.001" />
-        <origin xyz="0 0 0" rpy="0 0 0" />
-        <inertia ixx="0.00000015" ixy="0" ixz="0" iyy="0.00000015" iyz="0" izz="0.00000015" />
-    </inertial>
-</link>
-<joint name="imu_sensor_joint" type="fixed">
-    <axis xyz="0 0 1" />
-    <origin xyz="0 0 0" rpy="0 0 0" />
-    <parent link="chassis" />
-    <child link="imu_sensor_link" />
-</joint>
-<gazebo reference="imu_sensor_link">
-    <gravity>true</gravity>
-    <sensor name='imu_sensor' type='imu'>
-        <always_on>1</always_on>
-        <update_rate>30</update_rate>
-        <visualize>1</visualize>
-        <topic>__default_topic__</topic>
-        <plugin name='imu_plugin' filename='libgazebo_ros_imu_sensor.so'>
-    <frameName>imu_sensor_link</frameName>
-    <robotNamespace>/adabot</robotNamespace>
-            <topicName>imu_data</topicName>
-            <!-- <bodyName>imu_sensor_link</bodyName> -->
-            <updateRateHZ>30.0</updateRateHZ>
-            <gaussianNoise>0.0</gaussianNoise>
-            <xyzOffset>0 0 0</xyzOffset>
-            <rpyOffset>0 0 0</rpyOffset>
-        </plugin>
-        <pose>0 0 0 0 0 0</pose>
-    </sensor>
-</gazebo>
 </robot>

File: adabot_description/urdf/adabot.main.xacro (robot description, xacro)
@@ -4,4 +4,4 @@
     <xacro:include filename="$(find adabot_description)/urdf/macros/adabot.xacro" />
     <!-- Create an adabot -->
-    <xacro:adabot />
+    <xacro:adabot bot_name="a01" />
 </robot>

File: adabot_description/urdf/adabot.parameters.xacro (robot description, xacro)
@@ -18,6 +18,7 @@
          Properties for the robot bodies
     -->
-    <xacro:property name="PI" value="3.1415926535897931 " />
-    <xacro:property name="SCALE" value="$(arg scale)" />
+    <xacro:property name="PI"       value="3.1415926535897931 " />
+    <xacro:property name="SCALE"    value="$(arg scale)" />
+    <xacro:property name="MM_to_M"  value="0.001" />
     <!-- Typical density of plastics -->
     <xacro:property name="mat_density" value="1000.0" />
@@ -39,4 +40,7 @@
     <xacro:property name="wh_length"  value="${0.005 * SCALE}" />
     <xacro:property name="wh_mass"    value="${wh_density * PI * (wh_radius**2) * wh_length}" />
+    <!-- Wheel-Chassis joint parameters -->
+    <xacro:property name="wh_jnt_effort"    value="10" />
+    <xacro:property name="wh_jnt_velocity"  value="10" />
     <!-- Weg parameters -->
     <xacro:property name="ax_radius" value="${$(arg ax_radius) * SCALE}" />
@@ -48,4 +52,8 @@
     <xacro:property name="wg_mass"      value="${wg_density * wg_length * wg_width * wg_height}" />
     <xacro:property name="wg_per_wheel" value="$(arg wg_per_wheel)" />
+    <!-- Weg-Wheel joint parameters -->
+    <xacro:property name="wg_jnt_lower_limit"   value="0" />
+    <xacro:property name="wg_jnt_effort"        value="100" />
+    <xacro:property name="wg_jnt_velocity"      value="10" />
     <!-- Weg tip parameters -->
     <xacro:property name="wt_density_factor" value="0.5" />

File: adabot_description/urdf/macros/adabot.chassis.xacro (robot description, xacro)
@@ -8,7 +8,11 @@
         </geometry>
     </xacro:property>
-    <!-- Macro -->
+    <!--
+        Macro for creating chassis
+            chassis_name:   name used for the chasis link
+    -->
     <xacro:macro name="chassis" params="chassis_name">
-        <xacro:gz_white_material name="chassis" />
+        <!-- Add the roll cage's Gazebo material -->
+        <xacro:gz_white_material name="${chassis_name}" />
         <link name="${chassis_name}">
             <visual>
@@ -20,5 +24,5 @@
                     <geometry>
                         <mesh filename="package://adabot_description/meshes/chassis.stl"
-                              scale="${0.001 * SCALE} ${0.001 * SCALE} ${0.001 * SCALE}" />
+                              scale="${MM_to_M * SCALE} ${MM_to_M * SCALE} ${MM_to_M * SCALE}" />
                     </geometry>
                 </xacro:if>

File: adabot_description/urdf/macros/adabot.rollcage.xacro (robot description, xacro)
@@ -8,5 +8,8 @@
         </geometry>
     </xacro:property>
-    <!-- Macro -->
+    <!--
+        Macro for creating a roll cage
+            roll_cage_name: name used for the roll_care link
+    -->
     <xacro:macro name="roll_cage" params="roll_cage_name">
         <link name="${roll_cage_name}">

File: adabot_description/urdf/macros/adabot.weg.xacro (robot description, xacro)
@@ -18,10 +18,9 @@
             wheel  : the suffix of the parent wheel
             number : a unique identifier for each weg
-            parent : the full name of the parent link
             total  : the number of wegs (used to calculate angles)
     -->
-    <xacro:macro name="weg" params="wheel number parent total">
+    <xacro:macro name="weg" params="wheel number total bot_name">
         <!-- The name of the current weg (based on the parent wheel's name) -->
-        <xacro:property name="weg_name" value="${wheel}_weg_${number}" />
+        <xacro:property name="weg_name" value="${bot_name}_${wheel}_weg_${number}" />
         <!-- Add the weg's Gazebo material -->
         <xacro:gz_white_material name="${weg_name}" />
@@ -39,5 +38,5 @@
                     <geometry>
                         <mesh filename="package://adabot_description/meshes/weg.stl"
-                                scale="${0.001 * SCALE} ${0.001 * SCALE} ${0.001 * SCALE}" />
+                                scale="${MM_to_M * SCALE} ${MM_to_M * SCALE} ${MM_to_M * SCALE}" />
                     </geometry>
                 </xacro:if>
@@ -59,11 +58,4 @@
             </inertial>
         </link>
-        <!-- Connect the weg to the wheel with a prismatic joint -->
-        <joint name="${weg_name}_joint" type="prismatic">
-            <parent link="${parent}" />
-            <child link="${weg_name}" />
-            <origin xyz="0 0 0" rpy="0 ${2 * PI * (number/total)} 0" />
-            <limit upper="${wg_length}" lower="0" effort="100" velocity="10" />
-        </joint>
         <!--
              Attach a POSITION controller to each weg prismatic joint

File: adabot_description/urdf/macros/adabot.wheel.xacro (robot description, xacro)
@@ -12,7 +12,7 @@
             suffix     : give the wheel a unique name
     -->
-    <xacro:macro name="wheel" params="suffix">
+    <xacro:macro name="wheel" params="suffix bot_name">
         <!-- The name of the current wheel -->
-        <xacro:property name="wheel_name" value="${suffix}_wheel" />
+        <xacro:property name="wheel_name" value="${bot_name}_${suffix}_wheel" />
         <!-- Add the wheel's Gazebo material -->
         <xacro:gz_black_material name="${wheel_name}" />
@@ -29,5 +29,5 @@
                     <geometry>
                         <mesh filename="package://adabot_description/meshes/wheel.stl"
-                                scale="${0.001 * SCALE} ${0.001 * SCALE} ${0.001 * SCALE}" />
+                                scale="${MM_to_M * SCALE} ${MM_to_M * SCALE} ${MM_to_M * SCALE}" />
                     </geometry>
                 </xacro:if>
@@ -66,30 +66,50 @@
         </transmission>
         <!-- Add wegs to this wheel -->
+        <!-- Macro for weg-wheel joint -->
+        <xacro:macro name="weg_wheel_joint" params="weg_name number">
+            <joint name="${weg_name}_joint" type="prismatic">
+                <parent link="${wheel_name}" />
+                <child link="${weg_name}" />
+                <origin xyz="0 0 0" rpy="0 ${2 * PI * (number/wg_per_wheel)} 0" />
+                <limit upper="${wg_length}" lower="${wg_jnt_lower_limit}"
+                        effort="${wg_jnt_effort}" velocity="${wg_jnt_velocity}" />
+            </joint>
+        </xacro:macro>
+        <!-- Add the appropriate number of wegs -->
         <xacro:if value="${wg_per_wheel > 0}">
-            <xacro:weg wheel="${suffix}" number="1" parent="${wheel_name}" total="${wg_per_wheel}" />
+            <xacro:weg wheel="${suffix}" number="1" total="${wg_per_wheel}" bot_name="${bot_name}" />
+            <xacro:weg_wheel_joint weg_name="${bot_name}_${suffix}_weg_1" number="1" />
         </xacro:if>
         <xacro:if value="${wg_per_wheel > 1}">
-            <xacro:weg wheel="${suffix}" number="2" parent="${wheel_name}" total="${wg_per_wheel}" />
+            <xacro:weg wheel="${suffix}" number="2" total="${wg_per_wheel}" bot_name="${bot_name}" />
+            <xacro:weg_wheel_joint weg_name="${bot_name}_${suffix}_weg_2" number="2" />
         </xacro:if>
         <xacro:if value="${wg_per_wheel > 2}">
-            <xacro:weg wheel="${suffix}" number="3" parent="${wheel_name}" total="${wg_per_wheel}" />
+            <xacro:weg wheel="${suffix}" number="3" total="${wg_per_wheel}" bot_name="${bot_name}" />
+            <xacro:weg_wheel_joint weg_name="${bot_name}_${suffix}_weg_3" number="3" />
         </xacro:if>
         <xacro:if value="${wg_per_wheel > 3}">
-            <xacro:weg wheel="${suffix}" number="4" parent="${wheel_name}" total="${wg_per_wheel}" />
+            <xacro:weg wheel="${suffix}" number="4" total="${wg_per_wheel}" bot_name="${bot_name}" />
+            <xacro:weg_wheel_joint weg_name="${bot_name}_${suffix}_weg_4" number="4" />
         </xacro:if>
         <xacro:if value="${wg_per_wheel > 4}">
-            <xacro:weg wheel="${suffix}" number="5" parent="${wheel_name}" total="${wg_per_wheel}" />
+            <xacro:weg wheel="${suffix}" number="5" total="${wg_per_wheel}" bot_name="${bot_name}" />
+            <xacro:weg_wheel_joint weg_name="${bot_name}_${suffix}_weg_5" number="5" />
         </xacro:if>
         <xacro:if value="${wg_per_wheel > 5}">
-            <xacro:weg wheel="${suffix}" number="6" parent="${wheel_name}" total="${wg_per_wheel}" />
+            <xacro:weg wheel="${suffix}" number="6" total="${wg_per_wheel}" bot_name="${bot_name}" />
+            <xacro:weg_wheel_joint weg_name="${bot_name}_${suffix}_weg_6" number="6" />
         </xacro:if>
         <xacro:if value="${wg_per_wheel > 6}">
-            <xacro:weg wheel="${suffix}" number="7" parent="${wheel_name}" total="${wg_per_wheel}" />
+            <xacro:weg wheel="${suffix}" number="7" total="${wg_per_wheel}" bot_name="${bot_name}" />
+            <xacro:weg_wheel_joint weg_name="${bot_name}_${suffix}_weg_7" number="7" />
         </xacro:if>
         <xacro:if value="${wg_per_wheel > 7}">
-            <xacro:weg wheel="${suffix}" number="8" parent="${wheel_name}" total="${wg_per_wheel}" />
+            <xacro:weg wheel="${suffix}" number="8" total="${wg_per_wheel}" bot_name="${bot_name}" />
+            <xacro:weg_wheel_joint weg_name="${bot_name}_${suffix}_weg_8" number="8" />
         </xacro:if>
         <xacro:if value="${wg_per_wheel > 8}">
-            <xacro:weg wheel="${suffix}" number="9" parent="${wheel_name}" total="${wg_per_wheel}" />
+            <xacro:weg wheel="${suffix}" number="9" total="${wg_per_wheel}" bot_name="${bot_name}" />
+            <xacro:weg_wheel_joint weg_name="${bot_name}_${suffix}_weg_9" number="9" />
         </xacro:if>
     </xacro:macro>

File: adabot_description/urdf/macros/adabot.xacro (robot description, xacro)
@@ -9,48 +9,58 @@
     <!-- Include macros for creating all links and joints -->
     <xacro:include filename="$(find adabot_description)/urdf/macros/adabot.chassis.xacro" />
+    <xacro:include filename="$(find adabot_description)/urdf/macros/adabot.rollcage.xacro" />
+    <xacro:include filename="$(find adabot_description)/urdf/macros/adabot.imusensor.xacro" />
     <xacro:include filename="$(find adabot_description)/urdf/macros/adabot.wheel.xacro" />
     <xacro:include filename="$(find adabot_description)/urdf/macros/adabot.weg.xacro" />
-    <xacro:include filename="$(find adabot_description)/urdf/macros/adabot.rollcage.xacro" />
     <!-- Macro -->
-    <xacro:macro name="adabot">
+    <xacro:macro name="adabot" params="bot_name">
         <!-- Add a base_link to help with positioning -->
-        <link name="base_link" />
+        <link name="${bot_name}_base_link" />
         <!-- Add the chassis to the base_link -->
-        <xacro:chassis chassis_name="chassis"/>
-        <joint name="base_link_joint" type="fixed">
+        <xacro:property name="chassis_name" value="${bot_name}_chassis" />
+        <xacro:chassis chassis_name="${chassis_name}"/>
+        <joint name="${bot_name}_base_link_joint" type="fixed">
             <origin xyz="0 0 ${z_offset}" rpy="0 0 0" />
-            <parent link="base_link" />
-            <child link="chassis" />
+            <parent link="${bot_name}_base_link" />
+            <child link="${chassis_name}" />
         </joint>
         <!-- Add a roll cage to the chassis -->
-        <xacro:roll_cage roll_cage_name="roll_cage"/>
-        <joint name="chassis_cage_joint" type="fixed">
+        <xacro:roll_cage roll_cage_name="${bot_name}_roll_cage"/>
+        <joint name="${bot_name}_chassis_cage_joint" type="fixed">
             <origin xyz="0 0 ${cg_radius}" rpy="0 0 0" />
-            <parent link="chassis" />
-            <child link="roll_cage" />
+            <parent link="${chassis_name}" />
+            <child link="${bot_name}_roll_cage" />
+        </joint>
+        <!-- Add an imu sensor to the chassis -->
+        <xacro:imu_sensor bot_name="${bot_name}" />
+        <joint name="${bot_name}_imu_sensor_joint" type="fixed">
+            <axis xyz="0 0 1" />
+            <origin xyz="0 0 0" rpy="0 0 0" />
+            <parent link="${chassis_name}" />
+            <child link="${bot_name}_imu_sensor" />
         </joint>
         <!-- Add the wheels (note, wegs are created with the wheels) -->
         <!-- Wheel joint macro -->
         <xacro:macro name="wheel_joint" params="wheel_name reflect_fr reflect_lr">
-            <joint name="${wheel_name}_joint" type="continuous">
-                <parent link="chassis" />
+            <joint name="${bot_name}_${wheel_name}_joint" type="continuous">
+                <parent link="${chassis_name}" />
                 <child link="${wheel_name}" />
                 <origin xyz="${ch_length/2*reflect_fr} ${(wh_length+ch_width)/2*reflect_lr} 0" rpy="0 0 0" />
                 <axis xyz="0 1 0" />
-                <limit effort="10" velocity="10" />
+                <limit effort="${wh_jnt_effort}" velocity="${wh_jnt_velocity}" />
             </joint>
         </xacro:macro>
         <!--Front Left Wheel-->
-        <xacro:wheel suffix="front_left" />
-        <xacro:wheel_joint wheel_name="front_left_wheel" reflect_lr="1"  reflect_fr="1" />
+        <xacro:wheel suffix="front_left" bot_name="${bot_name}" />
+        <xacro:wheel_joint wheel_name="${bot_name}_front_left_wheel" reflect_lr="1"  reflect_fr="1" />
         <!--Front Right Wheel-->
-        <xacro:wheel suffix="front_right" />
-        <xacro:wheel_joint wheel_name="front_right_wheel" reflect_lr="-1"  reflect_fr="1" />
+        <xacro:wheel suffix="front_right" bot_name="${bot_name}" />
+        <xacro:wheel_joint wheel_name="${bot_name}_front_right_wheel" reflect_lr="-1"  reflect_fr="1" />
         <!--Rear Left Wheel-->
-        <xacro:wheel suffix="rear_left" />
-        <xacro:wheel_joint wheel_name="rear_left_wheel" reflect_lr="1"  reflect_fr="-1" />
+        <xacro:wheel suffix="rear_left" bot_name="${bot_name}" />
+        <xacro:wheel_joint wheel_name="${bot_name}_rear_left_wheel" reflect_lr="1"  reflect_fr="-1" />
         <!--Rear Right Wheel-->
-        <xacro:wheel suffix="rear_right" />
-        <xacro:wheel_joint wheel_name="rear_right_wheel" reflect_lr="-1"  reflect_fr="-1" />
+        <xacro:wheel suffix="rear_right" bot_name="${bot_name}" />
+        <xacro:wheel_joint wheel_name="${bot_name}_rear_right_wheel" reflect_lr="-1"  reflect_fr="-1" />
     </xacro:macro>
 </robot>
